File: doc/kicad/glycon.kicad_pcb (KiCad board)
At the start: 2 copper layers, 200 x 100 mm, 39 parts, among them IC1 SIO0-DIP-40, IC2 CTC-DIP-28, J1 Arduino/system bus header, J2 PMOD USBUART conn, J3 Int order hdr, J4 Conn_02x21_Odd_Even, SW1 SW_Push_Open, U0 Z80CPU, U1 628128_DIP32_SSOP32, U10 74HC244, U11 PIO-DIP-40, U12 74LS21, U2 SST39SF010, U3 74HC32, U4 74HC04, U6 74LS139, U7 SIO0-DIP-40, U9 74HC244, X1 ACO-6.00MHz

Commit message: more pcb work
Parts:
- removed the C7 at (125.0, 65.5)
- removed the C7 at (149.1, 152.3)
- removed IC1: SIO0-DIP-40, Package_DIP:DIP-40_W15.24mm_Socket
- removed U12: 74LS21, Package_DIP:DIP-14_W7.62mm_Socket
- added C12: 100nF, Capacitor_THT:C_Disc_D4.7mm_W2.5mm_P5.00mm, F.Cu at (145.9, 83.8)
- added C13: 100nF, Capacitor_THT:C_Disc_D4.7mm_W2.5mm_P5.00mm, F.Cu at (178.9, 83.7)
- added C7: 100nF, Capacitor_THT:C_Disc_D4.7mm_W2.5mm_P5.00mm, F.Cu at (36.1, 71.0)
- added U5: 74LS21, Package_DIP:DIP-14_W7.62mm_Socket, F.Cu at (114.8, 92.6)
- added U8: PIO-DIP-40, Package_DIP:DIP-40_W15.24mm_Socket, F.Cu at (61.6, 50.8)
- moved C10 177.3 mm to (69.7, 31.7), turned to -90 degrees
- moved U6 150.4 mm to (74.8, 38.0), turned to 90 degrees
- moved C11 127.0 mm to (72.2, 86.2), turned to 180 degrees
- moved C9 115.2 mm to (163.7, 109.1), turned to 90 degrees
- moved R3 86.1 mm to (105.9, 26.6), turned to 180 degrees
- moved R4 85.6 mm to (108.5, 26.6)
- moved U10 77.8 mm to (183.4, 90.0), turned to 90 degrees
- moved C5 77.7 mm to (98.9, 31.7), turned to -90 degrees
- moved R5 71.6 mm to (128.1, 87.5), turned to -90 degrees
- moved U3 71.2 mm to (103.4, 38.0), turned to 90 degrees
- moved R7 69.2 mm to (111.3, 100.1), turned to 90 degrees
- moved U9 68.7 mm to (151.0, 90.0), turned to 90 degrees
- moved R2 64.8 mm to (105.9, 41.2)
- moved C8 63.7 mm to (100.8, 76.1), turned to 180 degrees
- moved R6 63.6 mm to (111.0, 41.2), turned to 0 degrees
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Connections:
- net Net-(U6B-O3) renamed /~{IO_EN1}
- IC2 pad 6: /CLK -> /~{IORD}
- J1 pad 1: VDD -> +5V
- J1 pad 6: unconnected-(J1-Pin_6) -> /CLK
- J2 pad 6: VCC -> /VIN
- J4 pad 1: VDD -> +5V
- J4 pad 15: VDD -> +5V
- J4 pad 17: /PA7 -> /PB7
- J4 pad 18: /PB0 -> /PA0
- J4 pad 19: /PA6 -> /PB6
- J4 pad 20: /PB1 -> /PA1
- J4 pad 21: /PA5 -> /PB5
- J4 pad 22: /PB2 -> /PA2
- J4 pad 23: /PA4 -> /PB4
- J4 pad 24: /PB3 -> /PA3
- J4 pad 25: /PA3 -> /PB3
- J4 pad 26: /PB4 -> /PA4
- J4 pad 27: /PA2 -> /PB2
- J4 pad 28: /PB5 -> /PA5
- J4 pad 29: /PA1 -> /PB1
- J4 pad 30: /PB6 -> /PA6
- J4 pad 31: /PA0 -> /PB0
- J4 pad 32: /PB7 -> /PA7
- J4 pad 36: /SERCLK -> /~{W}/~{RDYA}
- J4 pad 4: /RESET -> /VIN
- J4 pad 40: /~{W}/~{RDYA} -> /RXDA
- J4 pad 41: VDD -> +5V
- J4 pad 6: unconnected-(J4-Pin_6) -> /RESET
- R2 pad 1: /CLK -> /~{RD}
- U0 pad 21: /CLK -> /~{RD}
- U1 pad 30: /A18 -> /A17
- U11 pad 35: /CLK -> /~{IORD}
- U2 pad 22: unconnected-(U2-~{CE}) -> /A17
- U3 pad 2: /CLK -> /~{RD}
- U7 pad 12: unconnected-(U7-RXDA) -> /RXDA
- U7 pad 32: /CLK -> /~{IORD}
Routing:
- net /CLK: track 65.5 -> 357.3 mm, vias 0 -> 3
- net /D1: track 93.2 -> 305.0 mm, vias 0 -> 4
- net /~{IORQ}: track 0.00 -> 202.0 mm
- net /D0: track 135.7 -> 297.0 mm, vias 2 -> 3
- net /PGA1: track 0.00 -> 159.3 mm, vias 0 -> 1
- net /RAM/ROM OE: track 0.00 -> 152.1 mm, vias 0 -> 1
- net /PGA0: track 0.00 -> 150.8 mm
- net /A14: track 0.00 -> 149.1 mm, vias 0 -> 2
- net Net-(U11-~{CE}): track 0.00 -> 148.8 mm, vias 0 -> 1
- net /~{RESET}: track 0.00 -> 141.2 mm, vias 0 -> 3
- net /A17: track 0.00 -> 140.2 mm, vias 0 -> 2
- net Net-(U10-2OE): track 0.00 -> 138.1 mm
- net /D3: track 169.2 -> 304.1 mm, vias 1 -> 4
- net /A16: track 0.00 -> 133.1 mm, vias 0 -> 1
- net /D5: track 161.5 -> 293.7 mm, vias 1 -> 2
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Other:
- outline, holes or cut-outs redrawn

Commit message: pcb design
Connections:
- J1 pad 10: unconnected-(J1-Pin_10) -> /BUSACK
- J1 pad 16: /~{M1} -> unconnected-(J1-Pin_16)
- J1 pad 37: /BUSACK -> /~{INTIN}
- J1 pad 39: /~{INTIN} -> Net-(J1-Pin_39)
- J1 pad 8: unconnected-(J1-Pin_8) -> /~{M1}
- J4 pad 11: /CT1 -> /TO1
- J4 pad 17: /PB7 -> /PB6
- J4 pad 18: /PA0 -> /PB7
- J4 pad 19: /PB6 -> /PB4
- J4 pad 20: /PA1 -> /PB5
- J4 pad 21: /PB5 -> /PB2
- J4 pad 22: /PA2 -> /PB3
- J4 pad 23: /PB4 -> /PB0
- J4 pad 24: /PA3 -> /PB1
- J4 pad 25: /PB3 -> /PA1
- J4 pad 26: /PA4 -> /PA0
- J4 pad 27: /PB2 -> /PA3
- J4 pad 28: /PA5 -> /PA2
- J4 pad 29: /PB1 -> /PA5
- J4 pad 30: /PA6 -> /PA4
- J4 pad 31: /PB0 -> /PA7
- J4 pad 32: /PA7 -> /PA6
- J4 pad 5: /TO2 -> /CT2
- J4 pad 7: /CT2 -> /CT1
- J4 pad 9: /TO1 -> /TO2
- R7 pad 2: /~{INTIN} -> Net-(J1-Pin_39)
- U5 pad 2: /~{INTIN} -> Net-(J1-Pin_39)
- U5 pad 4: /~{INT} -> Net-(U5-Pad4)
- U5 pad 8: /~{INT} -> Net-(U5-Pad4)
Routing:
- net /~{RESET}: track 141.2 -> 395.8 mm
- net Net-(J1-Pin_39): track 0.00 -> 216.4 mm
- net /BUSRQ: track 0.00 -> 204.5 mm
- net Net-(U7-~{INT}): track 0.00 -> 189.2 mm
- net /~{IORD}: track 0.00 -> 185.7 mm, vias 0 -> 5
- net /~{M1}: track 142.8 -> 320.6 mm, vias 2 -> 6
- net Net-(U2-~{WE}): track 0.00 -> 135.5 mm, vias 0 -> 2
- net /IEI2: track 0.00 -> 129.8 mm
- net /IEO2: track 0.00 -> 124.3 mm
- net /~{IORQ}: track 202.0 -> 316.5 mm, vias 0 -> 2
- net /BUSACK: track 0.00 -> 73.2 mm, vias 0 -> 1
- net /IEI1: track 0.00 -> 69.7 mm, vias 0 -> 2
- net /RESET: track 111.3 -> 173.8 mm, vias 1 -> 4
- net /IEO1: track 0.00 -> 60.1 mm, vias 0 -> 2
- net Net-(U8-~{INT}): track 0.00 -> 55.4 mm, vias 0 -> 2
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
Commit message: pcb work
Parts:
- J4: footprint Connector_PinHeader_2.54mm:PinHeader_2x21_P2.54mm_Vertical -> Connector_PinSocket_2.54mm:PinSocket_2x21_P2.54mm_Vertical
- moved J4 2.92 mm to (81.4, 113.3)
Connections:
- J4 pad 1: +5V -> Earth
- J4 pad 10: /PC2 -> /TO2
- J4 pad 11: /TO1 -> /PC1
- J4 pad 12: /PC1 -> /TO1
- J4 pad 13: /CLK -> /PC0
- J4 pad 14: /PC0 -> /CLK
- J4 pad 15: +5V -> Earth
- J4 pad 16: Earth -> +5V
- J4 pad 17: /PB6 -> /PB7
- J4 pad 18: /PB7 -> /PB6
- J4 pad 19: /PB4 -> /PB5
- J4 pad 2: Earth -> +5V
- J4 pad 20: /PB5 -> /PB4
- J4 pad 21: /PB2 -> /PB3
- J4 pad 22: /PB3 -> /PB2
- J4 pad 23: /PB0 -> /PB1
- J4 pad 24: /PB1 -> /PB0
- J4 pad 25: /PA1 -> /PA0
- J4 pad 26: /PA0 -> /PA1
- J4 pad 27: /PA3 -> /PA2
- J4 pad 28: /PA2 -> /PA3
- J4 pad 29: /PA5 -> /PA4
- J4 pad 3: /CT3 -> /VIN
- J4 pad 30: /PA4 -> /PA5
- J4 pad 31: /PA7 -> /PA6
- J4 pad 32: /PA6 -> /PA7
- J4 pad 33: /~{RTSA} -> /TXDA
- J4 pad 34: /TXDA -> /~{RTSA}
- J4 pad 35: /~{CTSA} -> /~{W}/~{RDYA}
- J4 pad 36: /~{W}/~{RDYA} -> /~{CTSA}
- J4 pad 37: /~{DTRA} -> /SYNCA
- J4 pad 38: /SYNCA -> /~{DTRA}
- J4 pad 39: /~{DCDA} -> /RXDA
- J4 pad 4: /VIN -> /CT3
- J4 pad 40: /RXDA -> /~{DCDA}
- J4 pad 41: +5V -> Earth
- J4 pad 42: Earth -> +5V
- J4 pad 5: /CT2 -> /RESET
- J4 pad 6: /RESET -> /CT2
- J4 pad 7: /CT1 -> /PC3
- J4 pad 8: /PC3 -> /CT1
- J4 pad 9: /TO2 -> /PC2
Routing:
- net /IEO2: track 124.3 -> 126.8 mm
- net /~{M1}: track 320.6 -> 318.8 mm
- net /IEI2: track 129.8 -> 131.5 mm
- net /TXDA: track 32.8 -> 32.1 mm
- net /IEO3: track 33.1 -> 32.4 mm
- net /CLK: track 365.5 -> 365.2 mm, vias 4 -> 3

Commit message: finish pcb trace routing
Parts:
- added H1: MountingHole_Pad, MountingHole:MountingHole_3.2mm_M3_Pad, F.Cu at (219.5, 116.0)
- added H2: MountingHole_Pad, MountingHole:MountingHole_3.2mm_M3_Pad, F.Cu at (219.5, 24.0)
- added H3: MountingHole_Pad, MountingHole:MountingHole_3.2mm_M3_Pad, F.Cu at (27.5, 24.0)
- added H4: MountingHole_Pad, MountingHole:MountingHole_3.2mm_M3_Pad, F.Cu at (27.5, 116.0)
- added H5: MountingHole_Pad, MountingHole:MountingHole_3.2mm_M3_Pad, F.Cu at (123.0, 76.0)
- added Q1: IRF9540N, Package_TO_SOT_THT:TO-220-3_Vertical, F.Cu at (57.1, 41.0)
- added Q2: IRF9540N, Package_TO_SOT_THT:TO-220-3_Vertical, F.Cu at (57.1, 33.3)
- added R10: 10K, Resistor_THT:R_Axial_DIN0204_L3.6mm_D1.6mm_P5.08mm_Horizontal, F.Cu at (51.4, 27.9)
- added R11: 10K, Resistor_THT:R_Axial_DIN0204_L3.6mm_D1.6mm_P5.08mm_Horizontal, F.Cu at (214.2, 104.5)
- added R8: 1K, Resistor_THT:R_Axial_DIN0204_L3.6mm_D1.6mm_P5.08mm_Horizontal, F.Cu at (51.4, 41.3)
- added SW2: SW_Push, Button_Switch_THT:SW_PUSH_6mm, F.Cu at (204.9, 108.5)
- moved R1 8.91 mm to (214.2, 102.4), turned to 90 degrees
- moved SW1 5.79 mm to (204.9, 99.9)
- moved C1 5.04 mm to (137.2, 52.1), turned to 0 degrees
- moved J4 4.30 mm to (85.1, 111.1)
- moved J1 0.54 mm to (211.5, 74.3)
- moved U7 0.10 mm to (31.0, 50.8)
Connections:
- J1 pad 1: +5V -> Earth
- J1 pad 37: /~{INTIN} -> unconnected-(J1-Pin_37)
- J1 pad 39: Net-(J1-Pin_39) -> /~{INTIN}
- J1 pad 40: Earth -> +5V
- J2 pad 6: /VIN -> +5V
- J4 pad 3: /VIN -> unconnected-(J4-Pin_3)
- R7 pad 2: Net-(J1-Pin_39) -> /~{INTIN}
- U0 pad 17: VDD -> /~{NMI}
- U5 pad 2: Net-(J1-Pin_39) -> /~{INTIN}
Routing:
- net VDD: track 4.19 -> 633.1 mm, vias 0 -> 6
- net +5V: track 0.00 -> 322.2 mm, vias 0 -> 2
- net Net-(J1-Pin_39): track 216.4 -> 0.00 mm
- net /~{INTIN}: track 0.00 -> 215.8 mm
- net /~{NMI}: track 0.00 -> 111.2 mm, vias 0 -> 2
- net /PC2: track 110.5 -> 194.7 mm
- net Earth: track 0.00 -> 60.5 mm, vias 0 -> 20
- net /CLK: track 365.2 -> 377.3 mm
- net /~{M1}: track 318.8 -> 328.5 mm
- net /D4: track 288.2 -> 296.0 mm
- net Net-(Q1-D): track 0.00 -> 7.62 mm
- net /~{INT}: track 52.7 -> 60.2 mm
- net Net-(U6B-O2): track 57.6 -> 50.9 mm
- net /D0: track 301.6 -> 307.9 mm
- net Net-(Q1-G): track 0.00 -> 5.85 mm
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- added copper zone on B.Cu, net Earth
- added copper zone on F.Cu, net Earth
Other:
- outline, holes or cut-outs redrawn
