File: doc/kicad/glycon.kicad_sch (KiCad schematic)
At the start: 32 parts, among them IC1 SIO0-DIP-40, IC2 CTC-DIP-28, J1 Arduino/system bus header, J2 PMOD USBUART conn, J3 Int order hdr, J4 Conn_02x26_Odd_Even, SW1 SW_Push, U0 Z80CPU, U1 628128_DIP32_SSOP32, U2 SST39SF010, U3 74HC32, U4 74HC04, U5 74LS21, U6 74LS138, U7 PIO-DIP-40, U8 PIO-DIP-40, X1 ACO-6.00MHz

Commit message: more schematic work
Parts:
- removed IC1: SIO0-DIP-40, Package_DIP:DIP-40_W15.24mm_Socket, symbol Zilog_Z80_Peripherals:SIO0-DIP-40
- removed J4: Conn_02x26_Odd_Even, Connector_PinSocket_2.54mm:PinSocket_2x26_P2.54mm_Vertical, symbol Connector_Generic:Conn_02x26_Odd_Even
- removed SW1: SW_Push, Button_Switch_THT:SW_PUSH_6mm, symbol Switch:SW_Push
- removed unit 1 of U5
- removed U6: 74LS138, Package_DIP:DIP-16_W7.62mm_Socket, symbol 74xx:74LS138
- removed U7: PIO-DIP-40, Package_DIP:DIP-40_W15.24mm_Socket, symbol Zilog_Z80_Peripherals:PIO-DIP-40
- added C10, C11, C9: 100nF, Capacitor_THT:C_Disc_D4.7mm_W2.5mm_P5.00mm, symbol Device:C
- added J4: Conn_02x21_Odd_Even, Connector_PinHeader_2.54mm:PinHeader_2x21_P2.54mm_Vertical, symbol Connector_Generic:Conn_02x21_Odd_Even
- added R7: 10K, Resistor_THT:R_Axial_DIN0204_L3.6mm_D1.6mm_P5.08mm_Horizontal, symbol Device:R
- added SW1: SW_Push_Open, Button_Switch_THT:SW_PUSH_6mm, symbol Switch:SW_Push_Open
- added U10, U9: 74HC244, Package_DIP:DIP-20_W7.62mm_Socket, symbol 74xx:74HC244
- added U11: PIO-DIP-40, Package_DIP:DIP-40_W15.24mm_Socket, symbol Zilog_Z80_Peripherals:PIO-DIP-40
- added U12: 74LS21, Package_DIP:DIP-14_W7.62mm_Socket, symbol 74xx:74LS21
- added unit 3 of U4
- added U6: 74LS139, Package_DIP:DIP-16_W7.62mm_Socket, symbol 74xx:74LS139
- added U7: SIO0-DIP-40, Package_DIP:DIP-40_W15.24mm_Socket, symbol Zilog_Z80_Peripherals:SIO0-DIP-40
Connections:
- net RAM_PGA0 is gone; now on net A14: U1.3 (A14)
- net RAM_PGA1 is gone; now on net A15: U1.31 (A15)
- net ROM_PGA0 is gone; now on net A14: U2.29 (A14)
- net ROM_PGA1 is gone; now on net A15: U2.3 (A15)
- net ROM_PGA2 is gone; now on net A16: U2.2 (A16)
- net A0: now also U11.6 (B/~{A}), U7.34 (B/~{A})
- net A1: now also U11.5 (C/~{D}), U7.33 (C/~{D})
- net A14: now also U10.18 (1Y0), U10.3 (2Y0), U9.18 (1Y0), U9.3 (2Y0); no longer J1.31 (Pin_31)
- net A15: now also U10.16 (1Y1), U10.5 (2Y1), U9.16 (1Y1), U9.5 (2Y1); no longer J1.33 (Pin_33), U0.5 (A15), U1.30 (CS2), U2.22 (~{CE})
- net A2: now also U6.14 (A0)
- net A3: now also U6.13 (A1)
- net CLK: now also J4.13 (Pin_13), U11.25 (CLK), U11.35 (~{RD}), U6.9 (O3), U7.20 (Φ), U7.32 (~{RD}), U7.35 (~{CE})
- net CT1: now also J4.11 (Pin_11)
- net CT2: now also J4.7 (Pin_7)
- net CT3: now also J4.3 (Pin_3)
- net CTSB: now also U7.23 (~{CTSB})
- net D0: now also U11.2 (D7), U7.40 (D0)
- net D1: now also U11.3 (D6), U7.1 (D1)
- net D2: now also U11.38 (D5), U7.39 (D2)
- net D3: now also U11.39 (D4), U7.2 (D3)
- net D4: now also U11.40 (D3), U7.38 (D4)
- net D5: now also U11.1 (D2), U7.3 (D5)
- net D6: now also U11.20 (D1), U7.37 (D6)
- net D7: now also U11.19 (D0), U7.4 (D7)
- net Earth: now also C3.1, R1.2, C10.2, C11.2, C9.2, J4.16 (Pin_16), J4.2 (Pin_2), J4.42 (Pin_42), U10.10 (GND), U10.11 (2A3), U10.13 (2A2), U10.15 (2A1), U10.17 (2A0), U11.11 (GND), U6.8 (GND), U7.31 (GND), U9.10 (GND); no longer C3.2, U1.22 (~{CS1})
- net IEI1: now also U11.24 (IEI)
- net IEI2: now also U7.6 (IEI)
- net IEO1: now also U11.22 (IEO)
- net IEO2: now also U7.7 (IEO)
- net PA0: now also J4.31 (Pin_31)
- net PA1: now also J4.29 (Pin_29)
- net PA2: now also J4.27 (Pin_27)
- net PA3: now also J4.25 (Pin_25)
- net PA4: now also J4.23 (Pin_23)
- net PA5: now also J4.21 (Pin_21)
- net PA6: now also J4.19 (Pin_19)
- net PA7: now also J4.17 (Pin_17)
- net PB0: now also J4.18 (Pin_18)
- net PB1: now also J4.20 (Pin_20)
- net PB2: now also J4.22 (Pin_22)
- net PB3: now also J4.24 (Pin_24)
- net PB4: now also J4.26 (Pin_26)
- net PB5: now also J4.28 (Pin_28)
- net PB6: now also J4.30 (Pin_30)
- net PB7: now also J4.32 (Pin_32)
- net PC0: now also J4.14 (Pin_14), U11.34 (PB7)
- net PC1: now also J4.12 (Pin_12), U11.33 (PB6)
- net PC2: now also J4.10 (Pin_10), U11.32 (PB5)
- net PC3: now also J4.8 (Pin_8), U11.31 (PB4)
- net RTSB: now also U7.24 (~{RTSB})
- net RxDB: now also U7.28 (RXDB)
- net SERCLK: now also J4.36 (Pin_36), U7.13 (~{RXCA}), U7.14 (~{TXCA}), U7.27 (~{RxTxCB})
- net TO1: now also J4.9 (Pin_9)
- net TO2: now also J4.5 (Pin_5)
- net TxDB: now also U7.26 (TXDB)
- net VDD: now also C3.2, U1.22 (~{CS1}), C10.1, C11.1, C9.1, R7.1, U10.20 (VCC), U11.26 (VCC), U12.13, U12.9, U6.1 (E), U6.15 (E), U6.16 (VCC), U7.9 (+5V), U9.20 (VCC); no longer C3.1, J1.1 (Pin_1), R1.1
- net ~{INT}: now also U12.12, U12.8
- net ~{IORQ}: now also U11.36 (~{IORQ}), U7.36 (~{IORQ})
- net ~{M1}: now also U11.37 (~{M1}), U7.8 (~{M1})
- net at U5.9: now also U7.5 (~{INT})
- net at U5.13: now also U11.23 (~{INT})
- net ~{INTIN}: now reaches J1.39 (Pin_39)
- net ~{INTIN}: now also R7.2, U12.10
- net RESET: now reaches J1.4 (Pin_4)
- net RESET: now also J4.6 (Pin_6), U4.5
- net ~{RESET}: now reaches U0.26 (~{RESET})
- net ~{RESET}: now also IC2.17 (~{RESET}), R1.1, SW1.2 (B), U7.21 (~{RESET}); no longer R1.2
- net PGA0: now reaches U0.4 (A14)
- net PGA0: now also J1.31 (Pin_31), U6.3 (A1)
- net at IC2.16 (~{CE}): now also U6.11 (O1)
- net at U8.4 (~{CE}): now also U6.10 (O2)
- net RAM_PGA2 renamed A16
- net A16: now also U10.14 (1Y2), U10.7 (2Y2), U9.14 (1Y2), U9.7 (2Y2)
- net VCC renamed VIN
- net VIN: now also J4.4 (Pin_4)
- new net: U11.10 (PA4), U9.17 (2A0)
- new net: U11.12 (PA3), U9.8 (1A3)
- new net: U11.13 (PA2), U9.6 (1A2)
- new net: U11.14 (PA1), U9.4 (1A1)
- new net: U11.15 (PA0), U9.2 (1A0)
- new net: U10.2 (1A0), U11.27 (PB0)
- new net: U10.4 (1A1), U11.28 (PB1)
- new net: U10.6 (1A2), U11.29 (PB2)
- new net: U10.8 (1A3), U11.30 (PB3)
- new net: U11.4 (~{CE}), U6.12 (O0)
- new net: U11.7 (PA7), U9.11 (2A3)
- new net: U11.8 (PA6), U9.13 (2A2)
- new net: U11.9 (PA5), U9.15 (2A1)
- new net: SW1.1 (A), U4.6
- new net: U10.19 (2OE), U6.4 (O0)
- new net: U10.1 (1OE), U6.5 (O1)
- new net: U6.6 (O2), U9.19 (2OE)
- new net: U6.7 (O3), U9.1 (1OE)
- new net +5V: J1.1 (Pin_1), J4.1 (Pin_1), J4.15 (Pin_15), J4.41 (Pin_41)
- new net A17: U10.12 (1Y3), U10.9 (2Y3), U9.12 (1Y3), U9.9 (2Y3)
- new net A18: U1.30 (CS2)
- new net PGA1: J1.33 (Pin_33), U0.5 (A15), U6.2 (A0)
- new net SYNCA: J4.38 (Pin_38), U7.11 (~{SYNCA})
- new net TXDA: J4.34 (Pin_34), U7.15 (TXDA)
- new net ~{CTSA}: J4.35 (Pin_35), U7.18 (~{CTSA})
- new net ~{DCDA}: J4.39 (Pin_39), U7.19 (~{DCDA})
- new net ~{DTRA}: J4.37 (Pin_37), U7.16 (~{DTRA})
- new net ~{RTSA}: J4.33 (Pin_33), U7.17 (~{RTSA})
- new net ~{W}/~{RDYA}: J4.40 (Pin_40), U7.10 (~{W}/~{RDYA})
Other:
- note added: "(ignore the addres order for now,see separate pinout pdf)"
- note added: "I/O"
- note added: "I/O Header"
- note added: "Paged memory decoding"
- note removed: "(RAM/ROM select)"
- note removed: "(ignore the addres order for now, see separate pinout pdf)"
- moved on the sheet: C1, C2, C3, C8, IC2, J3, R1, R6, U2, X1

Commit message: more pcb work
Parts:
- added C12, C13: 100nF, Capacitor_THT:C_Disc_D4.7mm_W2.5mm_P5.00mm, symbol Device:C
- renumbered U12 to U5
Connections:
- net A18 is gone; now on net A17: U1.30 (CS2)
- net A17: now also U2.22 (~{CE})
- net CLK: now also J1.6 (Pin_6); no longer IC2.6 (~{RD}), R2.1, U0.21 (~{RD}), U11.35 (~{RD}), U3.2, U6.9 (O3), U7.32 (~{RD}), U7.35 (~{CE}), U8.35 (~{RD})
- net Earth: now also C12.2, C13.2
- net PA0: now also J4.18 (Pin_18); no longer J4.31 (Pin_31)
- net PA1: now also J4.20 (Pin_20); no longer J4.29 (Pin_29)
- net PA2: now also J4.22 (Pin_22); no longer J4.27 (Pin_27)
- net PA3: now also J4.24 (Pin_24); no longer J4.25 (Pin_25)
- net PA4: now also J4.26 (Pin_26); no longer J4.23 (Pin_23)
- net PA5: now also J4.28 (Pin_28); no longer J4.21 (Pin_21)
- net PA6: now also J4.30 (Pin_30); no longer J4.19 (Pin_19)
- net PA7: now also J4.32 (Pin_32); no longer J4.17 (Pin_17)
- net PB0: now also J4.31 (Pin_31); no longer J4.18 (Pin_18)
- net PB1: now also J4.29 (Pin_29); no longer J4.20 (Pin_20)
- net PB2: now also J4.27 (Pin_27); no longer J4.22 (Pin_22)
- net PB3: now also J4.25 (Pin_25); no longer J4.24 (Pin_24)
- net PB4: now also J4.23 (Pin_23); no longer J4.26 (Pin_26)
- net PB5: now also J4.21 (Pin_21); no longer J4.28 (Pin_28)
- net PB6: now also J4.19 (Pin_19); no longer J4.30 (Pin_30)
- net PB7: now also J4.17 (Pin_17); no longer J4.32 (Pin_32)
- net SERCLK: no longer J4.36 (Pin_36)
- net VDD: now also U5.1, U5.5, C12.1, C13.1; no longer U5.13, U5.9
- net ~{INTIN}: now also U5.2; no longer U5.10
- net ~{INT}: now also U5.4, U5.6; no longer U5.12, U5.8
- net ~{W}/~{RDYA}: now also J4.36 (Pin_36); no longer J4.40 (Pin_40)
- net RXDA: now reaches U7.12 (RXDA)
- net RXDA: now also J4.40 (Pin_40)
- new net ~{IORD}: IC2.6 (~{RD}), U11.35 (~{RD}), U7.32 (~{RD}), U8.35 (~{RD})
- new net ~{IO_EN1}: U6.9 (O3), U7.35 (~{CE})
- new net ~{RD}: R2.1, U0.21 (~{RD}), U3.2
Other:
- moved on the sheet: J2, J3, J4, R1, SW1, U4C, X1

Commit message: pcb design
Connections:
- net BUSACK: now also J1.10 (Pin_10); no longer J1.37 (Pin_37)
- net CT1: now also J4.7 (Pin_7); no longer J4.11 (Pin_11)
- net CT2: now also J4.5 (Pin_5); no longer J4.7 (Pin_7)
- net PA0: now also J4.26 (Pin_26); no longer J4.18 (Pin_18)
- net PA1: now also J4.25 (Pin_25); no longer J4.20 (Pin_20)
- net PA2: now also J4.28 (Pin_28); no longer J4.22 (Pin_22)
- net PA3: now also J4.27 (Pin_27); no longer J4.24 (Pin_24)
- net PA4: now also J4.30 (Pin_30); no longer J4.26 (Pin_26)
- net PA5: now also J4.29 (Pin_29); no longer J4.28 (Pin_28)
- net PA6: now also J4.32 (Pin_32); no longer J4.30 (Pin_30)
- net PA7: now also J4.31 (Pin_31); no longer J4.32 (Pin_32)
- net PB0: now also J4.23 (Pin_23); no longer J4.31 (Pin_31)
- net PB1: now also J4.24 (Pin_24); no longer J4.29 (Pin_29)
- net PB2: now also J4.21 (Pin_21); no longer J4.27 (Pin_27)
- net PB3: now also J4.22 (Pin_22); no longer J4.25 (Pin_25)
- net PB4: now also J4.19 (Pin_19); no longer J4.23 (Pin_23)
- net PB5: now also J4.20 (Pin_20); no longer J4.21 (Pin_21)
- net PB6: now also J4.17 (Pin_17); no longer J4.19 (Pin_19)
- net PB7: now also J4.18 (Pin_18); no longer J4.17 (Pin_17)
- net TO1: now also J4.11 (Pin_11); no longer J4.9 (Pin_9)
- net TO2: now also J4.9 (Pin_9); no longer J4.5 (Pin_5)
- net ~{INTIN}: now also J1.37 (Pin_37); no longer J1.39 (Pin_39), R7.2, U5.2
- net ~{INT}: no longer U5.4, U5.8
- net ~{M1}: now also J1.8 (Pin_8); no longer J1.16 (Pin_16)
- new net: J1.39 (Pin_39), R7.2, U5.2
- new net: U5.4, U5.8

Commit message: pcb work
Parts:
- J4: footprint Connector_PinHeader_2.54mm:PinHeader_2x21_P2.54mm_Vertical -> Connector_PinSocket_2.54mm:PinSocket_2x21_P2.54mm_Vertical
Connections:
- net +5V: now also J4.16 (Pin_16), J4.2 (Pin_2), J4.42 (Pin_42); no longer J4.1 (Pin_1), J4.15 (Pin_15), J4.41 (Pin_41)
- net CLK: now also J4.14 (Pin_14); no longer J4.13 (Pin_13)
- net CT1: now also J4.8 (Pin_8); no longer J4.7 (Pin_7)
- net CT2: now also J4.6 (Pin_6); no longer J4.5 (Pin_5)
- net CT3: now also J4.4 (Pin_4); no longer J4.3 (Pin_3)
- net Earth: now also J4.1 (Pin_1), J4.15 (Pin_15), J4.41 (Pin_41); no longer J4.16 (Pin_16), J4.2 (Pin_2), J4.42 (Pin_42)
- net PA0: now also J4.25 (Pin_25); no longer J4.26 (Pin_26)
- net PA1: now also J4.26 (Pin_26); no longer J4.25 (Pin_25)
- net PA2: now also J4.27 (Pin_27); no longer J4.28 (Pin_28)
- net PA3: now also J4.28 (Pin_28); no longer J4.27 (Pin_27)
- net PA4: now also J4.29 (Pin_29); no longer J4.30 (Pin_30)
- net PA5: now also J4.30 (Pin_30); no longer J4.29 (Pin_29)
- net PA6: now also J4.31 (Pin_31); no longer J4.32 (Pin_32)
- net PA7: now also J4.32 (Pin_32); no longer J4.31 (Pin_31)
- net PB0: now also J4.24 (Pin_24); no longer J4.23 (Pin_23)
- net PB1: now also J4.23 (Pin_23); no longer J4.24 (Pin_24)
- net PB2: now also J4.22 (Pin_22); no longer J4.21 (Pin_21)
- net PB3: now also J4.21 (Pin_21); no longer J4.22 (Pin_22)
- net PB4: now also J4.20 (Pin_20); no longer J4.19 (Pin_19)
- net PB5: now also J4.19 (Pin_19); no longer J4.20 (Pin_20)
- net PB6: now also J4.18 (Pin_18); no longer J4.17 (Pin_17)
- net PB7: now also J4.17 (Pin_17); no longer J4.18 (Pin_18)
- net PC0: now also J4.13 (Pin_13); no longer J4.14 (Pin_14)
- net PC1: now also J4.11 (Pin_11); no longer J4.12 (Pin_12)
- net PC2: now also J4.9 (Pin_9); no longer J4.10 (Pin_10)
- net PC3: now also J4.7 (Pin_7); no longer J4.8 (Pin_8)
- net RESET: now also J4.5 (Pin_5); no longer J4.6 (Pin_6)
- net RXDA: now also J4.39 (Pin_39); no longer J4.40 (Pin_40)
- net SYNCA: now also J4.37 (Pin_37); no longer J4.38 (Pin_38)
- net TO1: now also J4.12 (Pin_12); no longer J4.11 (Pin_11)
- net TO2: now also J4.10 (Pin_10); no longer J4.9 (Pin_9)
- net TXDA: now also J4.33 (Pin_33); no longer J4.34 (Pin_34)
- net VIN: now also J4.3 (Pin_3); no longer J4.4 (Pin_4)
- net ~{CTSA}: now also J4.36 (Pin_36); no longer J4.35 (Pin_35)
- net ~{DCDA}: now also J4.40 (Pin_40); no longer J4.39 (Pin_39)
- net ~{DTRA}: now also J4.38 (Pin_38); no longer J4.37 (Pin_37)
- net ~{RTSA}: now also J4.34 (Pin_34); no longer J4.33 (Pin_33)
- net ~{W}/~{RDYA}: now also J4.35 (Pin_35); no longer J4.36 (Pin_36)
Other:
- moved on the sheet: U3A, U3B, U3C, U3D, U5A, U5B
Changed lines of the file:
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@@
     (pin "1")
   )
-  (symbol (lib_id "Connector_Generic:Conn_02x21_Odd_Even") (at 157.48 217.17 0) (unit 1)
+  (symbol (lib_id "Connector_Generic:Conn_02x21_Odd_Even") (at 160.02 217.17 0) (mirror y) (unit 1)
     (in_bom yes) (on_board yes) (fields_autoplaced)
     (property "Reference" "J4" (id 0) (at 158.75 186.69 0)
@@
       (effects (font (size 1.27 1.27)))
     )
-    (property "Footprint" "Connector_PinHeader_2.54mm:PinHeader_2x21_P2.54mm_Vertical" (id 2) (at 157.48 217.17 0)
-      (effects (font (size 1.27 1.27)) hide)
-    )
-    (property "Datasheet" "~" (id 3) (at 157.48 217.17 0)
+    (property "Footprint" "Connector_PinSocket_2.54mm:PinSocket_2x21_P2.54mm_Vertical" (id 2) (at 160.02 217.17 0)
+      (effects (font (size 1.27 1.27)) hide)
+    )
+    (property "Datasheet" "~" (id 3) (at 160.02 217.17 0)
       (effects (font (size 1.27 1.27)) hide)
     )
@@
     )
     (path "/eca3d929-6117-4a33-859d-45da5284422f"
-      (reference "J4") (unit 1) (value "Conn_02x21_Odd_Even") (footprint "Connector_PinHeader_2.54mm:PinHeader_2x21_P2.54mm_Vertical")
+      (reference "J4") (unit 1) (value "Conn_02x21_Odd_Even") (footprint "Connector_PinSocket_2.54mm:PinSocket_2x21_P2.54mm_Vertical")
     )
     (path "/bb31a07d-38a2-477f-a179-71f7c37ec131"

Commit message: finish pcb trace routing
Parts:
- added H1, H2, H3, H4, H5: MountingHole_Pad, MountingHole:MountingHole_3.2mm_M3_Pad, symbol Mechanical:MountingHole_Pad
- added Q1, Q2: IRF9540N, Package_TO_SOT_THT:TO-220-3_Vertical, symbol Transistor_FET:IRF9540N
- added R10, R11: 10K, Resistor_THT:R_Axial_DIN0204_L3.6mm_D1.6mm_P5.08mm_Horizontal, symbol Device:R
- added R8: 1K, Resistor_THT:R_Axial_DIN0204_L3.6mm_D1.6mm_P5.08mm_Horizontal, symbol Device:R
- added SW2: SW_Push, Button_Switch_THT:SW_PUSH_6mm, symbol Switch:SW_Push
Connections:
- net +5V: now also J1.40 (Pin_40), J2.6 (Pin_6), Q1.3 (S); no longer J1.1 (Pin_1)
- net Earth: now also J1.1 (Pin_1), H1.1, H2.1, H3.1, H4.1, H5.1, R10.1, R8.2, SW2.1; no longer J1.40 (Pin_40)
- net VDD: now also Q2.3 (S), R11.1; no longer U0.17 (~{NMI})
- net ~{INTIN}: now also J1.39 (Pin_39), R7.2, U5.2; no longer J1.37 (Pin_37)
- net VIN: no longer names the net of J4.3 (Pin_3)
- net VIN: no longer J2.6 (Pin_6)
- new net: Q2.1 (G), R10.2
- new net: Q1.2 (D), Q2.2 (D)
- new net: Q1.1 (G), R8.1
- new net ~{NMI}: R11.2, SW2.2, U0.17 (~{NMI})
Other:
- note added: "Reverse polarity protection"
- note removed: "Add some reverse polarity protection here"

Commit message: pcb refinement
Parts:
- removed J3: Int order hdr, Connector_PinHeader_2.54mm:PinHeader_2x06_P2.54mm_Vertical, symbol Connector_Generic:Conn_02x06_Odd_Even
- removed J4: Conn_02x21_Odd_Even, Connector_PinSocket_2.54mm:PinSocket_2x21_P2.54mm_Vertical, symbol Connector_Generic:Conn_02x21_Odd_Even
- removed SW1: SW_Push_Open, Button_Switch_THT:SW_PUSH_6mm, symbol Switch:SW_Push_Open
- added D1: LED, LED_THT:LED_D5.0mm, symbol Device:LED
- added J3: Conn_01x02, Connector_PinHeader_2.54mm:PinHeader_1x02_P2.54mm_Vertical, symbol Connector_Generic:Conn_01x02
- added J4: Conn_02x24_Odd_Even, Connector_PinSocket_2.54mm:PinSocket_2x24_P2.54mm_Vertical, symbol Connector_Generic:Conn_02x24_Odd_Even
- added R12: 470, Resistor_THT:R_Axial_DIN0204_L3.6mm_D1.6mm_P5.08mm_Horizontal, symbol Device:R
- added SW1: SW_Push, Button_Switch_THT:SW_PUSH_6mm, symbol Switch:SW_Push
- X1: value ACO-6.00MHz -> ACO-6.144MHz
- renumbered IC2 to U12
Connections:
- net IEO0 is gone; now on net VDD: U12.11 (IEO)
- net IEO1 is gone; now on net IEI0: U11.22 (IEO)
- net IEO2 is gone; now on net IEI1: U7.7 (IEO)
- net IEO3 is gone; now on net IEI2: U8.22 (IEO)
- net +5V: now also J4.1 (Pin_1), J4.15 (Pin_15), J4.37 (Pin_37), J4.47 (Pin_47)
- net CLK: now also J4.13 (Pin_13)
- net CT1: now also J4.7 (Pin_7)
- net CT2: now also J4.5 (Pin_5)
- net CT3: now also J4.3 (Pin_3)
- net Earth: now also U11.16 (~{ASTB}), U11.17 (~{BSTB}), U11.18 (ARDY), U11.21 (BRDY), J4.16 (Pin_16), J4.2 (Pin_2), J4.38 (Pin_38), J4.48 (Pin_48), R12.2
- net IEI3: now also J3.2 (Pin_2)
- net PA0: now also J4.30 (Pin_30)
- net PA1: now also J4.29 (Pin_29)
- net PA2: now also J4.32 (Pin_32)
- net PA3: now also J4.31 (Pin_31)
- net PA4: now also J4.34 (Pin_34)
- net PA5: now also J4.33 (Pin_33)
- net PA6: now also J4.36 (Pin_36)
- net PA7: now also J4.35 (Pin_35)
- net PB0: now also J4.23 (Pin_23)
- net PB1: now also J4.24 (Pin_24)
- net PB2: now also J4.21 (Pin_21)
- net PB3: now also J4.22 (Pin_22)
- net PB4: now also J4.19 (Pin_19)
- net PB5: now also J4.20 (Pin_20)
- net PB6: now also J4.17 (Pin_17)
- net PB7: now also J4.18 (Pin_18)
- net PC0: now also J4.14 (Pin_14)
- net PC1: now also J4.12 (Pin_12)
- net PC2: now also J4.10 (Pin_10)
- net PC3: now also J4.8 (Pin_8)
- net RESET: now also R1.1, J4.6 (Pin_6), SW1.1
- net RXDA: now also J4.46 (Pin_46)
- net SYNCA: now also J4.44 (Pin_44)
- net TO1: now also J4.11 (Pin_11)
- net TO2: now also J4.9 (Pin_9)
- net TXDA: now also J4.40 (Pin_40)
- net VDD: now also D1.2 (A), J3.1 (Pin_1), SW1.2
- net ~{CTSA}: now also J4.41 (Pin_41)
- net ~{DCDA}: now also J4.45 (Pin_45)
- net ~{DTRA}: now also J4.43 (Pin_43)
- net ~{RESET}: now also U4.6; no longer R1.1
- net ~{RTSA}: now also J4.39 (Pin_39)
- net ~{W}/~{RDYA}: now also J4.42 (Pin_42)
- net ~{ASTB}: now reaches U8.16 (~{ASTB})
- net ~{ASTB}: now also J4.27 (Pin_27)
- net ~{BSTB}: now reaches U8.17 (~{BSTB})
- net ~{BSTB}: now also J4.25 (Pin_25)
- net ~{ARDY}: now reaches U8.18 (ARDY)
- net ~{ARDY}: now also J4.28 (Pin_28)
- net ~{BRDY}: now reaches U8.21 (BRDY)
- net ~{BRDY}: now also J4.26 (Pin_26)
- new net: D1.1 (K), R12.1
Other:
- moved on the sheet: R11, SW2, U3A, U3B, U3C, U3D, U4C, U5A, U5B
