File: doc/kicad/_autosave-glycon.kicad_sch (KiCad schematic)
At the start: 56 parts, among them IC2 CTC-DIP-28, J1 Arduino/system bus header, J2 PMOD USBUART conn, J3 Int order hdr, J4 Conn_02x21_Odd_Even, Q1 IRF9540N, Q2 IRF9540N, SW2 SW_Push, U0 Z80CPU, U1 628128_DIP32_SSOP32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

Commit message: minor schematic updates
Parts:
- removed R2, R3, R4, R6: 10K, Resistor_THT:R_Axial_DIN0204_L3.6mm_D1.6mm_P5.08mm_Horizontal, symbol Device:R
- added RN1: 10K, Resistor_THT:R_Array_SIP10, symbol Device:R_Network09_Split
- gave numbers to parts that had none: 3
Connections:
- net Earth: now also RN1.1 (R1.1), RN1.3 (R2.2)
- net RAM/ROM OE: now also RN1.4 (R3.2)
- net ~{IORD}: now also RN1.2 (R1.2)
- net at U0.19 (~{MREQ}), U3.1, U3.12: now also RN1.5 (R4.2)
