File: doc/ledmatrix/ledmatrix.kicad_sch (KiCad schematic)
At the start: 183 parts, among them J1 Conn_01x04, Q1 2N2219, Q10 2N2219, Q11 2N2219, Q2 2N2219, Q3 2N2219, Q4 2N2219, Q5 2N2219, Q6 2N2219, Q7 2N2219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

Commit message: add BOM
Parts:
- R14: footprint (none) -> Resistor_THT:R_Axial_DIN0207_L6.3mm_D2.5mm_P7.62mm_Horizontal
Changed lines of the file:
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@@
       (effects (font (size 1.27 1.27)) (justify right))
     )
-    (property "Footprint" "" (id 2) (at 142.748 175.26 90)
+    (property "Footprint" "Resistor_THT:R_Axial_DIN0207_L6.3mm_D2.5mm_P7.62mm_Horizontal" (id 2) (at 142.748 175.26 90)
       (effects (font (size 1.27 1.27)) hide)
     )
@@
     )
     (path "/d3318490-1137-4881-bb77-fc7848f27e89"
-      (reference "R14") (unit 1) (value "470") (footprint "")
+      (reference "R14") (unit 1) (value "470") (footprint "Resistor_THT:R_Axial_DIN0207_L6.3mm_D2.5mm_P7.62mm_Horizontal")
     )
     (path "/9d4ac918-5702-45cc-aa2f-9d61f2ac5d34"
