File: hardware/kicad/glycon.kicad_pcb (KiCad board)
At the start: 2 copper layers, 200 x 100 mm, 59 parts, among them IC2 CTC-DIP-28, J1 Arduino/system bus header, J2 PMOD USBUART conn, J3 Conn_02x24_Odd_Even, J4 Conn_01x02, J5 USB_B, Q1 IRF9540N, Q2 IRF9540N, SW1 SW_Push, SW2 SW_Push, U0 Z80CPU, U1 628128_DIP32_SSOP32, U10 74HC244, U11 PIO-DIP-40, U2 SST39SF010, U3 74HC32, U4 74HC04, U5 74LS08, U6 74LS139, U7 SIO0-DIP-40, U8 PIO-DIP-40, U9 74HC244, X1 ACO-6.144MHz

Commit message: new PCB layout and initial routing
Parts:
- removed the H1 at (219.5, 116.0)
- removed the H1 at (27.5, 24.0)
- removed the H2 at (219.5, 116.0)
- removed the H2 at (219.5, 24.0)
- removed the H3 at (27.5, 116.0)
- removed the H3 at (27.5, 24.0)
- removed the H4 at (123.0, 76.0)
- removed the H4 at (27.5, 116.0)
- removed the H5 at (123.0, 76.0)
- removed the H5 at (219.5, 24.0)
- removed J5: USB_B, Connector_USB:USB_B_Lumberg_2411_02_Horizontal
- removed the R1 at (214.6, 99.7)
- removed the R1 at (123.6, 168.8)
- removed the R11 at (143.6, 150.6)
- removed the R11 at (221.0, 100.3)
- removed the R13 at (162.2, 159.5)
- removed the R5 at (147.3, 131.2)
- removed the R5 at (142.6, 171.1)
- removed the R9 at (137.4, 141.6)
- removed the R9 at (104.6, 152.1)
- removed RN1: 10K, Resistor_THT:R_Array_SIP10
- removed U4: 74HC04, Package_DIP:DIP-14_W7.62mm_Socket
- added C14: 100nF, Capacitor_THT:C_Disc_D4.7mm_W2.5mm_P5.00mm, F.Cu at (89.7, 142.0)
- added D2: LED, LED_THT:LED_D5.0mm, F.Cu at (161.2, 52.0)
- added D3: LED, LED_THT:LED_D5.0mm, F.Cu at (161.3, 58.5)
- added D4: LED, LED_THT:LED_D5.0mm, F.Cu at (161.3, 65.0)
- added D5: LED, LED_THT:LED_D5.0mm, F.Cu at (161.3, 71.5)
- added H1: MountingHole_Pad, MountingHole:MountingHole_3.2mm_M3_Pad, F.Cu at (160.0, 24.0)
- added H2: MountingHole_Pad, MountingHole:MountingHole_3.2mm_M3_Pad, F.Cu at (76.0, 127.6)
- added H3: MountingHole_Pad, MountingHole:MountingHole_3.2mm_M3_Pad, F.Cu at (267.0, 24.0)
- added H4: MountingHole_Pad, MountingHole:MountingHole_3.2mm_M3_Pad, F.Cu at (267.0, 131.0)
- added H5: MountingHole_Pad, MountingHole:MountingHole_3.2mm_M3_Pad, F.Cu at (160.0, 131.0)
- added R1: 10K, Resistor_THT:R_Axial_DIN0207_L6.3mm_D2.5mm_P10.16mm_Horizontal, F.Cu at (168.1, 113.0)
- added R10: 10K, Resistor_THT:R_Axial_DIN0207_L6.3mm_D2.5mm_P10.16mm_Horizontal, F.Cu at (87.8, 72.0)
- added R11: 10K, Resistor_THT:R_Axial_DIN0207_L6.3mm_D2.5mm_P10.16mm_Horizontal, F.Cu at (158.0, 89.0)
- added R13: 10K, Resistor_THT:R_Axial_DIN0207_L6.3mm_D2.5mm_P10.16mm_Horizontal, F.Cu at (87.8, 84.2)
- added R13: 470, Resistor_THT:R_Axial_DIN0207_L6.3mm_D2.5mm_P10.16mm_Horizontal, F.Cu at (158.0, 86.0)
- added R14: 10K, Resistor_THT:R_Axial_DIN0207_L6.3mm_D2.5mm_P10.16mm_Horizontal, F.Cu at (87.8, 88.2)
- added R15: 10K, Resistor_THT:R_Axial_DIN0207_L6.3mm_D2.5mm_P10.16mm_Horizontal, F.Cu at (88.9, 108.0)
- added R16: 10K, Resistor_THT:R_Axial_DIN0207_L6.3mm_D2.5mm_P10.16mm_Horizontal, F.Cu at (87.8, 96.3)
- added R17: 10K, Resistor_THT:R_Axial_DIN0207_L6.3mm_D2.5mm_P10.16mm_Horizontal, F.Cu at (87.8, 100.4)
- added R18: 10K, Resistor_THT:R_Axial_DIN0207_L6.3mm_D2.5mm_P10.16mm_Horizontal, F.Cu at (87.8, 104.5)
- added R19: 470, Resistor_THT:R_Axial_DIN0207_L6.3mm_D2.5mm_P10.16mm_Horizontal, F.Cu at (158.0, 83.0)
- added R2: 10K, Resistor_THT:R_Axial_DIN0207_L6.3mm_D2.5mm_P10.16mm_Horizontal, F.Cu at (126.8, 127.0)
- added R20: 470, Resistor_THT:R_Axial_DIN0207_L6.3mm_D2.5mm_P10.16mm_Horizontal, F.Cu at (158.0, 80.0)
- added R21: 470, Resistor_THT:R_Axial_DIN0207_L6.3mm_D2.5mm_P10.16mm_Horizontal, F.Cu at (158.0, 77.0)
- added R3: 10K, Resistor_THT:R_Axial_DIN0207_L6.3mm_D2.5mm_P10.16mm_Horizontal, F.Cu at (87.8, 43.7)
- added R4: 10K, Resistor_THT:R_Axial_DIN0207_L6.3mm_D2.5mm_P10.16mm_Horizontal, F.Cu at (87.8, 47.8)
- added R5: 10K, Resistor_THT:R_Axial_DIN0207_L6.3mm_D2.5mm_P10.16mm_Horizontal, F.Cu at (268.6, 83.0)
- added R6: 10K, Resistor_THT:R_Axial_DIN0207_L6.3mm_D2.5mm_P10.16mm_Horizontal, F.Cu at (87.8, 55.9)
- added R8: 10K, Resistor_THT:R_Axial_DIN0207_L6.3mm_D2.5mm_P10.16mm_Horizontal, F.Cu at (87.8, 64.0)
- added R9: 10K, Resistor_THT:R_Axial_DIN0207_L6.3mm_D2.5mm_P10.16mm_Horizontal, F.Cu at (87.8, 68.0)
- J1: value Arduino/system bus header -> Conn_02x20_Odd_Even
- J2: value PMOD USBUART conn -> Conn_01x06
- J4: value Conn_01x02 -> USB_B; footprint Connector_PinHeader_2.54mm:PinHeader_1x02_P2.54mm_Vertical -> Connector_USB:USB_B_TE_5787834_Vertical
- U1: value 628128_DIP32_SSOP32 -> BS62LV1027
- X1: footprint Oscillator:Oscillator_DIP-14 -> Oscillator:Oscillator_DIP-8
- moved X1 179.3 mm to (257.9, 119.5)
- moved J2 169.9 mm to (184.0, 130.5), turned to 90 degrees
- moved J3 169.2 mm to (260.5, 130.5)
- moved U7 162.1 mm to (192.0, 69.9)
- moved U8 152.4 mm to (212.8, 69.9)
- moved IC2 146.3 mm to (235.3, 88.5)
- moved Q1 145.9 mm to (185.4, 124.0)
- moved Q2 144.6 mm to (196.5, 124.0)
- moved U5 143.6 mm to (259.2, 90.4)
- moved U3 140.2 mm to (235.4, 85.3)
- moved R7 116.9 mm to (87.8, 59.9)
- moved U6 112.4 mm to (186.3, 24.6), turned to -90 degrees
- moved C13 104.5 mm to (89.7, 137.9), turned to 0 degrees
- moved C5 103.7 mm to (81.5, 133.9), turned to 0 degrees
- moved U0 103.7 mm to (235.8, 24.6)
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Connections:
- net /~{IORD} renamed /~{IO_RD}
- net /~{IO_EN1} renamed /SIO_~{CE}
- net Net-(IC2-Pad16) renamed /CTC_~{CE}
- net Net-(RN1-Pad9) renamed /~{MREQ}
- net Net-(U0-Pad22) renamed /~{Z80_WR}
- net Net-(U11-Pad4) renamed /PIO0_~{CE}
- net Net-(U6-Pad10) renamed /PIO1_~{CE}
- C9 pad 1: VDD -> Earth
- C9 pad 2: Earth -> VDD
- IC2 pad 11: VDD -> /IE10
- IC2 pad 12: Net-(IC2-Pad12) -> /~{INT}
- IC2 pad 13: /IEI0 -> /IEI1
- J1 pad 2: /ROM WE -> /~{ROM_WE}
- J1 pad 35: /BUSRQ -> /~{BUSRQ}
- J1 pad 39: /~{INTIN} -> /~{INT}
- J4 pad 1: VDD -> +5V
- J4 pad 2: /IEI3 -> unconnected-(J4-D--Pad2)
- R7 pad 1: VDD -> /~{INT}
- R7 pad 2: /~{INTIN} -> VDD
- SW1 pad 1: VDD -> Earth
- SW1 pad 2: /RESET -> /~{RESET}
- U0 pad 25: Net-(U0-Pad25) -> /~{BUSRQ}
- U1 pad 24: /~{MEMRD} -> /~{MEM_RD}
- U1 pad 29: Net-(U1-Pad29) -> /~{RAM_WE}
- U10 pad 14: /A16 -> /A14
- U10 pad 18: /A14 -> /A16
- U10 pad 2: Net-(U10-Pad2) -> Net-(U10-1A0)
- U10 pad 3: /A14 -> /A16
- U10 pad 6: Net-(U10-Pad6) -> Net-(U10-1A2)
- U10 pad 7: /A16 -> /A14
- U11 pad 10: Net-(U11-Pad10) -> Net-(U11-PA4)
- U11 pad 13: Net-(U11-Pad13) -> Net-(U11-PA2)
- U11 pad 15: Net-(U11-Pad15) -> Net-(U11-PA0)
- U11 pad 22: /IEI0 -> unconnected-(U11-IEO-Pad22)
- U11 pad 23: Net-(IC2-Pad12) -> /~{INT}
- U11 pad 24: /IEI1 -> /IEI0
- U11 pad 27: Net-(U10-Pad2) -> Net-(U10-1A2)
- U11 pad 29: Net-(U10-Pad6) -> Net-(U10-1A0)
- U11 pad 8: Net-(U11-Pad8) -> Net-(U11-PA6)
- U2 pad 24: /~{MEMRD} -> /~{MEM_RD}
- U2 pad 31: Net-(U2-Pad31) -> /~{ROM_WE}
- U3 pad 10: Net-(U3-Pad10) -> (no net)
- U3 pad 11: Net-(U3-Pad10) -> Net-(U3-Pad11)
- U3 pad 4: /RAM/ROM OE -> (no net)
- U3 pad 5: Net-(U3-Pad3) -> (no net)
- U3 pad 6: /~{MEMRD} -> (no net)
- U3 pad 8: Net-(U1-Pad29) -> (no net)
- U3 pad 9: /RAM WE -> (no net)
- U5 pad 1: /~{INTIN} -> /RAM/ROM OE
- U5 pad 10: (no net) -> /~{RESET}
- U5 pad 2: Net-(IC2-Pad12) -> Net-(U3-Pad3)
- U5 pad 3: /~{INT} -> /~{MEM_RD}
- U5 pad 4: /~{M1} -> /RAM WE
- U5 pad 5: /~{RESET} -> Net-(U3-Pad11)
- U5 pad 6: /~{PIO_M1} -> /~{RAM_WE}
- U5 pad 8: (no net) -> /~{PIO_M1}
- U5 pad 9: (no net) -> /~{M1}
- U6 pad 2: /PGA1 -> /PGA0
- U6 pad 3: /PGA0 -> /PGA1
- U6 pad 6: Net-(U6-Pad6) -> Net-(U6A-O2)
- U6 pad 7: Net-(U6-Pad7) -> Net-(U6A-O3)
- U7 pad 5: Net-(IC2-Pad12) -> /~{INT}
- U8 pad 23: Net-(IC2-Pad12) -> /~{INT}
- U8 pad 24: /IEI3 -> VDD
- U9 pad 1: Net-(U6-Pad7) -> Net-(U6A-O2)
- U9 pad 13: Net-(U11-Pad8) -> Net-(U11-PA4)
- U9 pad 14: /A16 -> /A14
- U9 pad 17: Net-(U11-Pad10) -> Net-(U11-PA6)
- U9 pad 18: /A14 -> /A16
- U9 pad 19: Net-(U6-Pad6) -> Net-(U6A-O3)
- U9 pad 2: Net-(U11-Pad15) -> Net-(U11-PA2)
- U9 pad 3: /A14 -> /A16
- U9 pad 6: Net-(U11-Pad13) -> Net-(U11-PA0)
- U9 pad 7: /A16 -> /A14
Routing:
- net VDD: track 628.9 -> 35.4 mm, vias 6 -> 0
- net /A1: track 604.4 -> 61.1 mm, vias 6 -> 0
- net /CLK: track 389.2 -> 0.00 mm, vias 4 -> 0
- net /D5: track 396.3 -> 39.2 mm, vias 4 -> 0
- net +5V: track 342.4 -> 0.00 mm, vias 1 -> 0
- net /D3: track 379.3 -> 46.7 mm, vias 5 -> 0
- net /~{IORQ}: track 314.6 -> 0.00 mm, vias 2 -> 0
- net /~{M1}: track 306.8 -> 0.00 mm, vias 6 -> 0
- net /D1: track 340.3 -> 45.8 mm, vias 4 -> 0
- net /~{IO_RD}: track 245.5 -> 0.00 mm, vias 6 -> 0
- net /D4: track 292.5 -> 47.5 mm, vias 4 -> 0
- net /A0: track 299.8 -> 61.1 mm, vias 5 -> 0
- net /D7: track 241.6 -> 30.9 mm, vias 3 -> 2
- net /~{RESET}: track 199.5 -> 0.00 mm, vias 3 -> 0
- net /D6: track 226.4 -> 32.7 mm, vias 2 -> 0
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- removed copper zone on B.Cu, net Earth
- removed copper zone on F.Cu, net Earth
Other:
- board size 200 x 100 mm -> 115 x 115 mm
- board text added: "CTSA"
- board text added: "RAWE"
- board text added: "~{ASTB}"
- board text removed: "Arduino/expansion header"
- board text removed: "CTC"
- board text removed: "Glycon"
- board text removed: "IO Header"
- board text removed: "NMI"
- board text removed: "PIO 1"
- board text removed: "PIO 2"
- board text removed: "PWR"
- board text removed: "RAM"
- board text removed: "RESET"
- board text removed: "ROM"
- board text removed: "SIO"
- board text removed: "USBUART"
- board text removed: "Z80 CPU"

Commit message: kicad work
Parts:
- moved J3 59.6 mm to (201.0, 133.0), turned to 90 degrees
- moved Q2 40.7 mm to (155.9, 120.5), turned to 90 degrees
- moved Q1 24.2 mm to (161.4, 120.5), turned to 90 degrees
- moved U8 23.7 mm to (189.8, 75.8)
- moved U7 21.6 mm to (212.8, 75.8)
- moved R1 15.3 mm to (153.7, 107.8), turned to 0 degrees
- moved SW1 11.8 mm to (158.8, 97.5), turned to -90 degrees
- moved D3 11.4 mm to (156.8, 48.0)
- moved D4 11.4 mm to (156.8, 54.5)
- moved D5 11.4 mm to (156.8, 61.0)
- moved D2 11.4 mm to (156.8, 41.5)
- moved R11 7.91 mm to (163.9, 83.8), turned to 180 degrees
- moved D1 7.28 mm to (156.8, 127.5)
- moved U11 7.25 mm to (166.9, 75.8)
- moved H5 7.07 mm to (155.0, 136.0)
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Connections:
- IC2 pad 11: /IE10 -> /IEI0
- J3 pad 1: +5V -> Earth
- J3 pad 10: /PC2 -> /~{RTSA}
- J3 pad 11: /TO1 -> Earth
- J3 pad 12: /PC1 -> +5V
- J3 pad 13: /CLK -> /PA6
- J3 pad 14: /PC0 -> /PA7
- J3 pad 15: +5V -> /PA4
- J3 pad 16: Earth -> /PA5
- J3 pad 17: /PB6 -> /PA2
- J3 pad 18: /PB7 -> /PA3
- J3 pad 19: /PB4 -> /PA0
- J3 pad 2: Earth -> +5V
- J3 pad 20: /PB5 -> /PA1
- J3 pad 21: /PB2 -> /ARDY
- J3 pad 22: /PB3 -> /~{ASTB}
- J3 pad 23: /PB0 -> /BRDY
- J3 pad 24: /PB1 -> /~{BSTB}
- J3 pad 25: /~{BSTB} -> /PB1
- J3 pad 26: /BRDY -> /PB0
- J3 pad 27: /~{ASTB} -> /PB3
- J3 pad 28: /ARDY -> /PB2
- J3 pad 29: /PA1 -> /PB5
- J3 pad 3: /CT3 -> /RXDA
- J3 pad 30: /PA0 -> /PB4
- J3 pad 31: /PA3 -> /PB7
- J3 pad 32: /PA2 -> /PB6
- J3 pad 33: /PA5 -> Earth
- J3 pad 34: /PA4 -> +5V
- J3 pad 35: /PA7 -> /PC0
- J3 pad 36: /PA6 -> /CLK
- J3 pad 37: +5V -> /PC1
- J3 pad 38: Earth -> /TO1
- J3 pad 39: /~{RTSA} -> /PC2
- J3 pad 4: unconnected-(J3-Pin_4-Pad4) -> /~{DCDA}
- J3 pad 40: /TXDA -> /TO2
- J3 pad 41: /~{CTSA} -> /PC3
- J3 pad 42: /~{W}/~{RDYA} -> /CT1
- J3 pad 43: /~{DTRA} -> /RESET
- J3 pad 44: /SYNCA -> /CT2
- J3 pad 45: /~{DCDA} -> unconnected-(J3-Pin_45-Pad45)
- J3 pad 46: /RXDA -> /CT3
- J3 pad 47: +5V -> Earth
- J3 pad 48: Earth -> +5V
- J3 pad 5: /CT2 -> /SYNCA
- J3 pad 6: /RESET -> /~{DTRA}
- J3 pad 7: /CT1 -> /~{W}/~{RDYA}
- J3 pad 8: /PC3 -> /~{CTSA}
- J3 pad 9: /TO2 -> /TXDA
Routing:
- net /D2: track 50.9 -> 149.3 mm
- net /D3: track 46.7 -> 133.9 mm, vias 0 -> 2
- net /D7: track 30.9 -> 117.3 mm, vias 2 -> 3
- net /D6: track 32.7 -> 114.8 mm
- net /D1: track 45.8 -> 121.3 mm
- net Earth: track 5.57 -> 78.6 mm
- net /PC0: track 0.00 -> 72.1 mm, vias 0 -> 2
- net /D0: track 45.8 -> 114.5 mm
- net /D5: track 39.2 -> 106.1 mm, vias 0 -> 1
- net /PC1: track 0.00 -> 66.6 mm, vias 0 -> 2
- net /D4: track 47.5 -> 112.6 mm
- net /PC2: track 0.00 -> 61.0 mm, vias 0 -> 2
- net /PGA1: track 70.6 -> 13.9 mm
- net /PC3: track 0.00 -> 55.5 mm, vias 0 -> 2
- net /PIO0_~{CE}: track 0.00 -> 54.9 mm
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Other:
- board size 115 x 115 mm -> 120 x 120 mm

Commit message: More pcb progress
Parts:
- removed C4: 100nF, Capacitor_THT:C_Disc_D4.7mm_W2.5mm_P5.00mm
- removed R10, R14, R15, R16, R5, R6, R9: 10K, Resistor_THT:R_Axial_DIN0207_L6.3mm_D2.5mm_P10.16mm_Horizontal
- removed the R13 at (87.8, 84.2)
- added JP1: Jumper, Connector_PinHeader_2.54mm:PinHeader_2x01_P2.54mm_Vertical, F.Cu at (221.3, 71.5)
- added JP2: Jumper, Connector_PinHeader_2.54mm:PinHeader_2x01_P2.54mm_Vertical, F.Cu at (227.8, 71.5)
- moved C6 190.1 mm to (266.0, 92.0), turned to 180 degrees
- moved R3 184.5 mm to (268.1, 83.0), turned to 180 degrees
- moved C5 180.9 mm to (254.0, 79.5), turned to -90 degrees
- moved R4 174.3 mm to (257.9, 86.0)
- moved C14 173.1 mm to (260.5, 114.0)
- moved R8 171.9 mm to (257.9, 89.0)
- moved R2 147.7 mm to (260.0, 63.0), turned to -90 degrees
- moved H2 145.6 mm to (209.5, 69.5)
- moved C7 143.6 mm to (218.0, 97.5)
- moved C8 141.8 mm to (246.0, 101.0), turned to 180 degrees
- moved C10 137.3 mm to (184.0, 26.0), turned to -90 degrees
- moved C13 136.5 mm to (181.5, 37.0), turned to 180 degrees
- moved R7 127.8 mm to (180.4, 148.0)
- moved C12 125.9 mm to (170.0, 37.0), turned to 180 degrees
- moved C11 110.5 mm to (198.5, 111.0), turned to 180 degrees
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Connections:
- J1 pad 1: Earth -> /A17
- J1 pad 10: /~{BUSACK} -> /A8
- J1 pad 11: /A3 -> /A7
- J1 pad 12: /A16 -> /A6
- J1 pad 13: /A4 -> /A5
- J1 pad 14: /A15 -> /A4
- J1 pad 15: /A11 -> /A3
- J1 pad 16: /A14 -> /A2
- J1 pad 17: /A5 -> /A1
- J1 pad 18: /~{IORQ} -> /A0
- J1 pad 19: /A9 -> /D4
- J1 pad 2: /~{ROM_WE} -> /A16
- J1 pad 20: /RAM/ROM OE -> /D3
- J1 pad 21: /A6 -> /D5
- J1 pad 22: /RAM WE -> /D6
- J1 pad 23: /A8 -> /D2
- J1 pad 24: /D0 -> /D7
- J1 pad 25: /A7 -> /D0
- J1 pad 27: /A13 -> /~{RESET}
- J1 pad 28: /D2 -> /~{BUSRQ}
- J1 pad 29: /A12 -> /~{INT}
- J1 pad 3: /A0 -> /A15
- J1 pad 30: /D3 -> /~{BUSACK}
- J1 pad 31: /PGA0 -> /~{M1}
- J1 pad 32: /D4 -> unconnected-(J1-Pin_32-Pad32)
- J1 pad 33: /PGA1 -> unconnected-(J1-Pin_33-Pad33)
- J1 pad 34: /D5 -> unconnected-(J1-Pin_34-Pad34)
- J1 pad 35: /~{BUSRQ} -> /RAM WE
- J1 pad 36: /D6 -> /CLK
- J1 pad 37: /A14 -> /RAM/ROM OE
- J1 pad 38: /D7 -> /~{ROM_WE}
- J1 pad 39: /~{INT} -> Earth
- J1 pad 4: /RESET -> /A14
- J1 pad 40: +5V -> VDD
- J1 pad 5: /A1 -> /A13
- J1 pad 6: /CLK -> /A12
- J1 pad 7: /A2 -> /A11
- J1 pad 8: /~{M1} -> /A10
- J1 pad 9: /A10 -> /A9
- J2 pad 1: /RTSB -> +5V
- J2 pad 2: /RxDB -> Earth
- J2 pad 3: /TxDB -> /CTSB
- J2 pad 4: /CTSB -> /TxDB
- J2 pad 5: Earth -> /RxDB
- J2 pad 6: +5V -> /RTSB
- J3 pad 10: /~{RTSA} -> /PA1
- J3 pad 11: Earth -> /ARDY
- J3 pad 12: +5V -> /~{ASTB}
- J3 pad 13: /PA6 -> /PB6
- J3 pad 14: /PA7 -> /PB7
- J3 pad 15: /PA4 -> /PB4
- J3 pad 16: /PA5 -> /PB5
- J3 pad 17: /PA2 -> /PB2
- J3 pad 18: /PA3 -> /PB3
- J3 pad 19: /PA0 -> /PB0
- J3 pad 20: /PA1 -> /PB1
- J3 pad 21: /ARDY -> /BRDY
- J3 pad 22: /~{ASTB} -> /~{BSTB}
- J3 pad 23: /BRDY -> Earth
- J3 pad 24: /~{BSTB} -> +5V
- J3 pad 25: /PB1 -> /SYNCA
- J3 pad 26: /PB0 -> /~{W}/~{RDYA}
- J3 pad 27: /PB3 -> /TXDA
- J3 pad 28: /PB2 -> /RXDA
- J3 pad 29: /PB5 -> /~{RTSA}
- J3 pad 3: /RXDA -> /PA6
- J3 pad 30: /PB4 -> /~{DTRA}
- J3 pad 31: /PB7 -> /~{DCDA}
- J3 pad 32: /PB6 -> /~{CTSA}
- J3 pad 33: Earth -> unconnected-(J3-Pin_33-Pad33)
- J3 pad 34: +5V -> unconnected-(J3-Pin_34-Pad34)
- J3 pad 35: /PC0 -> /CLK
- J3 pad 36: /CLK -> unconnected-(J3-Pin_36-Pad36)
- J3 pad 37: /PC1 -> /TO1
- J3 pad 38: /TO1 -> unconnected-(J3-Pin_38-Pad38)
- J3 pad 39: /PC2 -> /TO2
- J3 pad 4: /~{DCDA} -> /PA7
- J3 pad 40: /TO2 -> unconnected-(J3-Pin_40-Pad40)
- J3 pad 41: /PC3 -> /CT1
- J3 pad 42: /CT1 -> unconnected-(J3-Pin_42-Pad42)
- J3 pad 43: /RESET -> /CT2
- J3 pad 44: /CT2 -> unconnected-(J3-Pin_44-Pad44)
- J3 pad 45: unconnected-(J3-Pin_45-Pad45) -> /CT3
- J3 pad 46: /CT3 -> unconnected-(J3-Pin_46-Pad46)
- J3 pad 5: /SYNCA -> /PA4
- J3 pad 6: /~{DTRA} -> /PA5
- J3 pad 7: /~{W}/~{RDYA} -> /PA2
- J3 pad 8: /~{CTSA} -> /PA3
- J3 pad 9: /TXDA -> /PA0
- R2 pad 1: /~{IO_RD} -> /~{BUSRQ}
- R3 pad 1: /~{Z80_WR} -> VDD
- R3 pad 2: VDD -> /~{ROM_WE}
- U0 pad 1: /A11 -> unconnected-(U0-A11-Pad1)
- U0 pad 10: /D6 -> /~{BUSRQ}
- U0 pad 12: /D2 -> /~{MREQ}
- U0 pad 13: /D7 -> /~{BUSACK}
- U0 pad 14: /D0 -> /~{IO_RD}
- U0 pad 15: /D1 -> /~{Z80_WR}
- U0 pad 16: /~{INT} -> /A7
- U0 pad 17: /~{NMI} -> /A6
- U0 pad 18: unconnected-(U0-~{HALT}-Pad18) -> /A13
- U0 pad 19: /~{MREQ} -> /D2
- U0 pad 2: /A12 -> VDD
- U0 pad 20: /~{IORQ} -> /D3
- U0 pad 21: /~{IO_RD} -> /D0
- U0 pad 22: /~{Z80_WR} -> /D1
- U0 pad 23: /~{BUSACK} -> /D7
- U0 pad 24: VDD -> /A12
- U0 pad 25: /~{BUSRQ} -> /D6
- U0 pad 26: /~{RESET} -> /A0
- U0 pad 27: /~{M1} -> /A10
- U0 pad 28: unconnected-(U0-~{RFSH}-Pad28) -> /A11
- U0 pad 3: /A13 -> unconnected-(U0-A13-Pad3)
- U0 pad 30: /A0 -> /~{RESET}
- U0 pad 31: /A1 -> unconnected-(U0-A1-Pad31)
- U0 pad 32: /A2 -> unconnected-(U0-A2-Pad32)
- U0 pad 33: /A3 -> /CLK
- U0 pad 34: /A4 -> unconnected-(U0-A4-Pad34)
- U0 pad 35: /A5 -> unconnected-(U0-A5-Pad35)
- U0 pad 36: /A6 -> /~{NMI}
- U0 pad 37: /A7 -> /~{INT}
- U0 pad 38: /A8 -> unconnected-(U0-A8-Pad38)
- U0 pad 39: /A9 -> unconnected-(U0-A9-Pad39)
- U0 pad 4: /PGA0 -> unconnected-(U0-A14-Pad4)
- U0 pad 40: /A10 -> /~{M1}
- U0 pad 5: /PGA1 -> unconnected-(U0-A15-Pad5)
- U0 pad 6: /CLK -> /A3
- U0 pad 7: /D4 -> unconnected-(U0-D4-Pad7)
- U0 pad 8: /D3 -> /~{IORQ}
- U0 pad 9: /D5 -> unconnected-(U0-D5-Pad9)
- U7 pad 13: /SERCLK -> Net-(JP2-B)
- U7 pad 14: /SERCLK -> Net-(JP1-B)
Routing:
- net /CLK: track 24.0 -> 256.5 mm, vias 0 -> 5
- net /~{RESET}: track 10.5 -> 212.9 mm, vias 0 -> 1
- net /~{PIO_M1}: track 23.8 -> 139.4 mm, vias 0 -> 1
- net /~{M1}: track 0.00 -> 107.3 mm, vias 0 -> 1
- net VDD: track 35.4 -> 111.7 mm
- net /~{NMI}: track 10.5 -> 76.4 mm
- net /PGA1: track 13.9 -> 76.6 mm, vias 1 -> 0
- net /PGA0: track 9.91 -> 70.1 mm
- net /PA7: track 0.00 -> 48.0 mm
- net /PB7: track 0.00 -> 47.1 mm
- net /A11: track 46.5 -> 92.4 mm
- net /A13: track 34.5 -> 78.9 mm
- net /~{INT}: track 24.1 -> 67.7 mm, vias 0 -> 2
- net /PA5: track 0.00 -> 43.4 mm
- net /~{W}/~{RDYA}: track 0.00 -> 42.9 mm
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Other:
- board text removed: "~{ASTB}"

Commit message: almost finalized new pcb design
Parts:
- added R5: 10K, Resistor_THT:R_Axial_DIN0207_L6.3mm_D2.5mm_P10.16mm_Horizontal, F.Cu at (215.3, 71.0)
- moved R7 87.3 mm to (215.3, 68.0)
- moved JP2 41.7 mm to (209.0, 108.8), turned to 90 degrees
- moved JP1 36.3 mm to (232.0, 106.2), turned to -90 degrees
- moved X1 7.38 mm to (265.3, 126.3), turned to 90 degrees
- moved C10 5.00 mm to (184.0, 31.0), turned to 90 degrees
- moved R2 4.36 mm to (255.6, 63.0)
- moved C11 0.90 mm to (197.6, 111.0)
- moved H2 0.71 mm to (209.0, 70.0)
- moved J2 0.50 mm to (260.7, 135.5)
- moved C12 0.50 mm to (170.0, 36.5)
- moved C13 0.50 mm to (181.5, 36.5)
- renumbered IC2 to U12
Connections:
- net /RTSB renamed /~{RTSB}
- J2 pad 1: +5V -> Earth
- J2 pad 2: Earth -> /~{CTSB}
- J2 pad 3: /CTSB -> +5V
- J3 pad 26: /~{W}/~{RDYA} -> unconnected-(J3-Pin_26-Pad26)
- J3 pad 33: unconnected-(J3-Pin_33-Pad33) -> Earth
- J3 pad 34: unconnected-(J3-Pin_34-Pad34) -> +5V
- J3 pad 36: unconnected-(J3-Pin_36-Pad36) -> /PC0
- J3 pad 38: unconnected-(J3-Pin_38-Pad38) -> /PC1
- J3 pad 40: unconnected-(J3-Pin_40-Pad40) -> /PC2
- J3 pad 42: unconnected-(J3-Pin_42-Pad42) -> /PC3
- U0 pad 1: unconnected-(U0-A11-Pad1) -> /A11
- U0 pad 10: /~{BUSRQ} -> /D6
- U0 pad 12: /~{MREQ} -> /D2
- U0 pad 13: /~{BUSACK} -> /D7
- U0 pad 14: /~{IO_RD} -> /D0
- U0 pad 15: /~{Z80_WR} -> /D1
- U0 pad 16: /A7 -> /~{INT}
- U0 pad 17: /A6 -> /~{NMI}
- U0 pad 18: /A13 -> unconnected-(U0-~{HALT}-Pad18)
- U0 pad 19: /D2 -> /~{MREQ}
- U0 pad 2: VDD -> /A12
- U0 pad 20: /D3 -> /~{IORQ}
- U0 pad 21: /D0 -> /~{IO_RD}
- U0 pad 22: /D1 -> /~{Z80_WR}
- U0 pad 23: /D7 -> /~{BUSACK}
- U0 pad 24: /A12 -> /~{WAIT}
- U0 pad 25: /D6 -> /~{BUSRQ}
- U0 pad 26: /A0 -> /~{RESET}
- U0 pad 27: /A10 -> /~{M1}
- U0 pad 28: /A11 -> unconnected-(U0-~{RFSH}-Pad28)
- U0 pad 3: unconnected-(U0-A13-Pad3) -> /A13
- U0 pad 30: /~{RESET} -> /A0
- U0 pad 31: unconnected-(U0-A1-Pad31) -> /A1
- U0 pad 32: unconnected-(U0-A2-Pad32) -> /A2
- U0 pad 33: /CLK -> /A3
- U0 pad 34: unconnected-(U0-A4-Pad34) -> /A4
- U0 pad 35: unconnected-(U0-A5-Pad35) -> /A5
- U0 pad 36: /~{NMI} -> /A6
- U0 pad 37: /~{INT} -> /A7
- U0 pad 38: unconnected-(U0-A8-Pad38) -> /A8
- U0 pad 39: unconnected-(U0-A9-Pad39) -> /A9
- U0 pad 4: unconnected-(U0-A14-Pad4) -> /PGA0
- U0 pad 40: /~{M1} -> /A10
- U0 pad 5: unconnected-(U0-A15-Pad5) -> /PGA1
- U0 pad 6: /A3 -> /CLK
- U0 pad 7: unconnected-(U0-D4-Pad7) -> /D4
- U0 pad 8: /~{IORQ} -> /D3
- U0 pad 9: unconnected-(U0-D5-Pad9) -> /D5
- U7 pad 10: /~{W}/~{RDYA} -> /~{WAIT}
- U7 pad 23: /CTSB -> /~{CTSB}
- U7 pad 30: unconnected-(U7-~{W}/~{RDYB}-Pad30) -> /~{WAIT}
- X1 pad 4: (no net) -> Earth
- X1 pad 5: (no net) -> /CLK
- X1 pad 8: /CLK -> VDD
Routing:
- net VDD: track 111.7 -> 536.7 mm, vias 0 -> 6
- net Earth: track 111.3 -> 452.6 mm, vias 0 -> 10
- net /CTC_~{CE}: track 0.00 -> 182.2 mm, vias 0 -> 2
- net /~{INT}: track 67.7 -> 194.6 mm, vias 2 -> 4
- net /SIO_~{CE}: track 0.00 -> 125.5 mm, vias 0 -> 2
- net /A1: track 104.1 -> 224.4 mm, vias 0 -> 2
- net /A0: track 100.3 -> 219.4 mm
- net /PC3: track 55.5 -> 163.9 mm
- net /D0: track 153.2 -> 257.5 mm, vias 0 -> 4
- net /PC0: track 72.1 -> 167.9 mm
- net /PC1: track 66.6 -> 161.7 mm
- net /PC2: track 61.0 -> 155.0 mm
- net /~{WAIT}: track 0.00 -> 90.4 mm, vias 0 -> 1
- net /~{IORQ}: track 23.8 -> 113.9 mm, vias 0 -> 4
- net +5V: track 22.8 -> 111.7 mm
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- added copper zone on B.Cu, net Earth
- added copper zone on F.Cu, net Earth
Other:
- board text added: "5V"
- board text added: "A0"
- board text added: "A1"
- board text added: "A10"
- board text added: "A11"
- board text added: "A12"
- board text added: "A13"
- board text added: "A14"
- board text added: "A15"
- board text added: "A16"
- board text added: "A17"
- board text added: "A2"
- board text added: "A3"
- board text added: "A4"
- board text added: "A5"
- board text added: "A6"
- board text added: "A7"
- board text added: "A8"
- board text added: "A9"
- board text added: "ARDY"
- board text added: "BRDY"
- board text added: "CLK"
- board text added: "CT1"
- board text added: "CT2"
- board text added: "CT3"
- board text added: "CTC"
- board text added: "D0"
- board text added: "D1"
- board text added: "D2"
- board text added: "D3"
- board text added: "D4"
- board text added: "D5"
- board text added: "D6"
- board text added: "D7"
- board text added: "GLYCON"
- board text added: "GND"
- board text added: "GPIO"
- board text added: "NC"
- board text added: "NMI"
- board text added: "PA0"
- board text added: "PA1"
- board text added: "PA2"
- board text added: "PA3"
- board text added: "PA4"
- board text added: "PA5"
- board text added: "PA6"
- board text added: "PA7"
- board text added: "PB0"
- board text added: "PB1"
- board text added: "PB2"
- board text added: "PB3"
- board text added: "PB4"
- board text added: "PB5"
- board text added: "PB6"
- board text added: "PB7"
- board text added: "PC0"
- board text added: "PC1"
- board text added: "PC2"
- board text added: "PC3"
- board text added: "PIO0"
- board text added: "PIO1"
- board text added: "PWR"
- board text added: "RAM"
- board text added: "RESET"
- board text added: "ROM"
- board text added: "RROE"
- board text added: "RXDA"
- board text added: "SIO"
- board text added: "SYNCA"
- board text added: "SYSTEM BUS HEADER"
- board text added: "TO1"
- board text added: "TO2"
- board text added: "TXDA"
- board text added: "UART"
- board text added: "VDD"
- board text added: "Z80 CPU"
- board text added: "Z80 Computer"
- board text added: "~{ASTB}"
- board text added: "~{BSACK}"
- board text added: "~{BSRQ}"
- board text added: "~{BTSB}"
- board text added: "~{CTSA}"
- board text added: "~{DCDA}"
- board text added: "~{DTRA}"
- board text added: "~{INT}"
- board text added: "~{M1}"
- board text added: "~{ROWE}"
- board text added: "~{RST}"
- board text added: "~{RTSA}"
