File: hardware/kicad/glycon.kicad_sch (KiCad schematic)
At the start: 59 parts, among them IC2 CTC-DIP-28, J1 Conn_02x20_Odd_Even, J2 Conn_01x06, J3 Conn_02x24_Odd_Even, Q1 IRF9540N, Q2 IRF9540N, SW1 SW_Push, SW2 SW_Push, U0 Z80CPU, U1 BS62LV1027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

Commit message: create pdf of revised schematic
Parts:
- added J4: USB_B, Connector_USB:USB_B_OST_USB-B1HSxx_Horizontal, symbol Connector:USB_B
Connections:
- net +5V: now also J4.1 (VBUS)
- net Earth: now also J4.4 (GND), J4.5 (Shield)
- no-connect marks 9 -> 16

Commit message: new PCB layout and initial routing
Parts:
- removed C4: 100nF, Capacitor_THT:C_Disc_D4.7mm_W2.5mm_P5.00mm, symbol Device:C
- removed unit 2 of U3
- removed unit 3 of U3
- removed U4: 74HC04, Package_DIP:DIP-14_W7.62mm_Socket, symbol 74xx:74HC04
- added D2, D3, D4, D5: LED, LED_THT:LED_D5.0mm, symbol Device:LED
- added R19, R20, R21: 470, Resistor_THT:R_Axial_DIN0207_L6.3mm_D2.5mm_P10.16mm_Horizontal, symbol Device:R
- added unit 2 of U5
- J4: footprint Connector_USB:USB_B_OST_USB-B1HSxx_Horizontal -> Connector_USB:USB_B_TE_5787834_Vertical
- R13: value 10K -> 470
- X1: footprint Oscillator:Oscillator_DIP-14 -> Oscillator:Oscillator_DIP-8
Connections:
- net BUSRQ is gone; now on net ~{BUSRQ}: J1.35 (Pin_35), R9.2
- net ROM WE is gone; now on net ~{ROM_WE}: J1.2 (Pin_2), R5.2
- net +5V: now also R5.1, R9.1
- net A14: now also U10.14 (1Y2), U10.7 (2Y2), U9.14 (1Y2), U9.7 (2Y2); no longer U10.18 (1Y0), U10.3 (2Y0), U9.18 (1Y0), U9.3 (2Y0)
- net A16: now also U10.18 (1Y0), U10.3 (2Y0), U9.18 (1Y0), U9.3 (2Y0); no longer U10.14 (1Y2), U10.7 (2Y2), U9.14 (1Y2), U9.7 (2Y2)
- net Earth: now also R13.2, SW1.1, R19.2, R20.2, R21.2; no longer R1.2, R2.2, R3.2, R4.2, R5.1, R6.2, R8.2, R9.1
- net PC0: now also D2.2 (A)
- net PC1: now also D3.2 (A)
- net PC2: now also D4.2 (A)
- net PC3: now also D5.2 (A)
- net RAM WE: now also U5.4
- net RAM/ROM OE: now also U5.1
- net RESET: no longer R1.1, SW1.2
- net VDD: now also R1.2, R2.2, R3.2, R4.2, R6.2, R8.2; no longer R13.2, SW1.1
- net ~{INT}: now also J1.39 (Pin_39), R7.1, U0.16 (~{INT}); no longer R13.1, U5.2
- net ~{M1}: now also U5.9; no longer U5.4
- net ~{MEM_RD}: now also U5.3
- net ~{PIO_M1}: now also U5.8; no longer U5.6
- net ~{RAM_WE}: now also U5.6
- net ~{RESET}: now also R1.1, SW1.2, U5.10; no longer U5.5
- net at U3.11: now also U5.5
- net at U11.10 (PA4): now also U9.13 (2A2); no longer U9.17 (2A0)
- net at U11.13 (PA2): now also U9.2 (1A0); no longer U9.6 (1A2)
- net at U11.15 (PA0): now also U9.6 (1A2); no longer U9.2 (1A0)
- net at U11.27 (PB0): now also U10.6 (1A2); no longer U10.2 (1A0)
- net at U11.29 (PB2): now also U10.2 (1A0); no longer U10.6 (1A2)
- net at U11.8 (PA6): now also U9.17 (2A0); no longer U9.13 (2A2)
- net at U3.3: now also U5.2
- removed net ~{INTIN}: J1.39 (Pin_39), R7.1, U5.1
- removed net ~{Z80_INT}: U0.16 (~{INT}), U5.3
- new net: D4.1 (K), R19.1
- new net: D2.1 (K), R21.1
- new net: D3.1 (K), R20.1
- new net: D5.1 (K), R13.1
Other:
- moved on the sheet: R1, R11, R5, SW1, SW2

Commit message: kicad work
Connections:
- net IE10 is gone; now on net IEI0: IC2.11 (IEO)
- net +5V: now also J3.12 (Pin_12), J3.2 (Pin_2), J3.34 (Pin_34), J3.48 (Pin_48); no longer J3.1 (Pin_1), J3.15 (Pin_15), J3.37 (Pin_37), J3.47 (Pin_47)
- net ARDY: now also J3.21 (Pin_21); no longer J3.28 (Pin_28)
- net BRDY: now also J3.23 (Pin_23); no longer J3.26 (Pin_26)
- net CLK: now also J3.36 (Pin_36); no longer J3.13 (Pin_13)
- net CT1: now also J3.42 (Pin_42); no longer J3.7 (Pin_7)
- net CT2: now also J3.44 (Pin_44); no longer J3.5 (Pin_5)
- net CT3: now also J3.46 (Pin_46); no longer J3.3 (Pin_3)
- net Earth: now also J3.1 (Pin_1), J3.11 (Pin_11), J3.33 (Pin_33), J3.47 (Pin_47); no longer J3.16 (Pin_16), J3.2 (Pin_2), J3.38 (Pin_38), J3.48 (Pin_48)
- net PA0: now also J3.19 (Pin_19); no longer J3.30 (Pin_30)
- net PA1: now also J3.20 (Pin_20); no longer J3.29 (Pin_29)
- net PA2: now also J3.17 (Pin_17); no longer J3.32 (Pin_32)
- net PA3: now also J3.18 (Pin_18); no longer J3.31 (Pin_31)
- net PA4: now also J3.15 (Pin_15); no longer J3.34 (Pin_34)
- net PA5: now also J3.16 (Pin_16); no longer J3.33 (Pin_33)
- net PA6: now also J3.13 (Pin_13); no longer J3.36 (Pin_36)
- net PA7: now also J3.14 (Pin_14); no longer J3.35 (Pin_35)
- net PB0: now also J3.26 (Pin_26); no longer J3.23 (Pin_23)
- net PB1: now also J3.25 (Pin_25); no longer J3.24 (Pin_24)
- net PB2: now also J3.28 (Pin_28); no longer J3.21 (Pin_21)
- net PB3: now also J3.27 (Pin_27); no longer J3.22 (Pin_22)
- net PB4: now also J3.30 (Pin_30); no longer J3.19 (Pin_19)
- net PB5: now also J3.29 (Pin_29); no longer J3.20 (Pin_20)
- net PB6: now also J3.32 (Pin_32); no longer J3.17 (Pin_17)
- net PB7: now also J3.31 (Pin_31); no longer J3.18 (Pin_18)
- net PC0: now also J3.35 (Pin_35); no longer J3.14 (Pin_14)
- net PC1: now also J3.37 (Pin_37); no longer J3.12 (Pin_12)
- net PC2: now also J3.39 (Pin_39); no longer J3.10 (Pin_10)
- net PC3: now also J3.41 (Pin_41); no longer J3.8 (Pin_8)
- net RESET: now also J3.43 (Pin_43); no longer J3.6 (Pin_6)
- net RXDA: now also J3.3 (Pin_3); no longer J3.46 (Pin_46)
- net SYNCA: now also J3.5 (Pin_5); no longer J3.44 (Pin_44)
- net TO1: now also J3.38 (Pin_38); no longer J3.11 (Pin_11)
- net TO2: now also J3.40 (Pin_40); no longer J3.9 (Pin_9)
- net TXDA: now also J3.9 (Pin_9); no longer J3.40 (Pin_40)
- net ~{ASTB}: now also J3.22 (Pin_22); no longer J3.27 (Pin_27)
- net ~{BSTB}: now also J3.24 (Pin_24); no longer J3.25 (Pin_25)
- net ~{CTSA}: now also J3.8 (Pin_8); no longer J3.41 (Pin_41)
- net ~{DCDA}: now also J3.4 (Pin_4); no longer J3.45 (Pin_45)
- net ~{DTRA}: now also J3.6 (Pin_6); no longer J3.43 (Pin_43)
- net ~{RTSA}: now also J3.10 (Pin_10); no longer J3.39 (Pin_39)
- net ~{W}/~{RDYA}: now also J3.7 (Pin_7); no longer J3.42 (Pin_42)
Changed lines of the file:
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@@
 		(exclude_from_sim no)
 		(at 43.18 239.395 0)
-		(size 33.655 8.255)
+		(size 33.655 10.795)
 		(stroke
 			(width 0)
@@
 		(exclude_from_sim no)
 		(at 136.525 203.2 0)
-		(size 39.37 13.97)
+		(size 39.37 16.51)
 		(stroke
 			(width 0)
@@
 	(text_box "The paged memory controller allows the Z80 to acces more than 64K of\nmemory. It is essentially 4 4-bit registers with a selectable output\nmask that allows the Z80 to select one of these at any moment to\ncontrol the upper four bits of the address bus (A14 through A17).\nThe registers are actually PIO ports (half of port A plus all of\nport B), plus one hardcoded register that always reads 0x0, which is\nthe default page, so that the Z80 can always find the bootcode.\n\nThe output mask is controlled by the upper two bits of the Z80 address\noutput, referred to as PGA0 and PGA1. The rest of the addres bits of\nthe z8 are connected directly to the memory chips. This results in the\nmemory map of the Z80 essentially being split into 4 blocks of 16K. \nThe upper four adress bits, so the output of the paged memory \ncontroller are connected to the memory chips too. A14 through A16 then\nselectdifferent areas of memory on the chips, and A17 selects between \nRAM and ROM. All this allows the Z80 to acces 256K of memory, 128K of \nRAM and 128K of ROM. "
 		(exclude_from_sim no)
-		(at 287.02 17.78 0)
-		(size 24.13 15.24)
+		(at 335.28 12.7 0)
+		(size 31.75 16.51)
 		(stroke
 			(width 0)
@@
 		(effects
 			(font
-				(size 0.508 0.508)
+				(size 0.5 0.5)
 			)
 			(justify left top)
@@
 		)
 	)
-	(label "IE10"
+	(label "IEI0"
 		(at 133.35 190.5 0)
 		(fields_autoplaced yes)
@@
 	)
 	(symbol
+		(lib_id "Connector_Generic:Conn_02x24_Odd_Even")
+		(at 382.27 208.28 180)
+		(unit 1)
+		(exclude_from_sim no)
+		(in_bom yes)
+		(on_board yes)
+		(dnp no)
+		(fields_autoplaced yes)
+		(property "Reference" "J3"
+			(at 381 171.45 0)
+			(effects
+				(font
+					(size 1.27 1.27)
+				)
+			)
+		)
+		(property "Value" "Conn_02x24_Odd_Even"
+			(at 381 173.99 0)
+			(effects
+				(font
+					(size 1.27 1.27)
+				)
+			)
+		)
+		(property "Footprint" "Connector_PinSocket_2.54mm:PinSocket_2x24_P2.54mm_Vertical"
+			(at 382.27 208.28 0)
+			(effects
+				(font
+					(size 1.27 1.27)
+				)
+				(hide yes)
+			)
+		)
+		(property "Datasheet" "~"
+			(at 382.27 208.28 0)
+			(effects
+				(font
+					(size 1.27 1.27)
+				)
+				(hide yes)
+			)
+		)
+		(property "Description" ""
+			(at 382.27 208.28 0)
+			(effects
+				(font
+					(size 1.27 1.27)
+				)
+				(hide yes)
+			)
+		)
+		(pin "1"
+		)
+		(pin "10"
+		)
+		(pin "11"
+		)
+		(pin "12"
+		)
+		(pin "13"
+		)
+		(pin "14"
+		)
+		(pin "15"
+		)
+		(pin "16"
+		)
+		(pin "17"
+		)
+		(pin "18"
+		)
+		(pin "19"
+		)
+		(pin "2"
+		)
+		(pin "20"
+		)
+		(pin "21"
+		)
+		(pin "22"
+		)
+		(pin "23"
+		)
+		(pin "24"
+		)
+		(pin "25"
+		)
+		(pin "26"
+		)
+		(pin "27"
+		)
+		(pin "28"
+		)
+		(pin "29"
+		)
+		(pin "3"
+		)
+		(pin "30"
+		)
+		(pin "31"
+		)
+		(pin "32"
+		)
+		(pin "33"
+		)
+		(pin "34"
+		)
+		(pin "35"
+		)
+		(pin "36"
+		)
+		(pin "37"
+		)
+		(pin "38"
+		)
+		(pin "39"
+		)
+		(pin "4"
+		)
+		(pin "40"
+		)
+		(pin "41"
+		)
+		(pin "42"
+		)
+		(pin "43"
+		)
+		(pin "44"
+		)
+		(pin "45"
+		)
+		(pin "46"
+		)
+		(pin "47"
+		)
+		(pin "48"
+		)
+		(pin "5"
+		)
+		(pin "6"
+		)
+		(pin "7"
+		)
+		(pin "8"
+		)
+		(pin "9"
+		)
+		(instances
+			(project "glycon"
+				(path "/956d8204-2614-4e68-9498-0bae56c4b641"
+					(reference "J3")
+					(unit 1)
+				)
+			)
+		)
+	)
+	(symbol
 		(lib_id "Memory_RAM:628128_DIP32_SSOP32")
 		(at 193.04 69.85 0)
@@
 					(unit 1)
 				)
-			)
-		)
-	)
-	(symbol
-		(lib_id "Connector_Generic:Conn_02x24_Odd_Even")
-		(at 379.73 205.74 0)
-		(unit 1)
-		(exclude_from_sim no)
-		(in_bom yes)
-		(on_board yes)
-		(dnp no)
-		(fields_autoplaced yes)
-		(property "Reference" "J3"
-			(at 381 171.45 0)
-			(effects
-				(font
-					(size 1.27 1.27)
-				)
-			)
-		)
-		(property "Value" "Conn_02x24_Odd_Even"
-			(at 381 173.99 0)
-			(effects
-				(font
-					(size 1.27 1.27)
-				)
-			)
-		)
-		(property "Footprint" "Connector_PinSocket_2.54mm:PinSocket_2x24_P2.54mm_Vertical"
-			(at 379.73 205.74 0)
-			(effects
-				(font
-					(size 1.27 1.27)
-				)
-				(hide yes)
-			)
-		)
-		(property "Datasheet" "~"
-			(at 379.73 205.74 0)
-			(effects
-				(font
-					(size 1.27 1.27)
-				)
-				(hide yes)
-			)
-		)
-		(property "Description" ""
-			(at 379.73 205.74 0)
-			(effects
-				(font
-					(size 1.27 1.27)
-				)
-				(hide yes)
-			)
-		)
-		(pin "1"
-		)
-		(pin "10"
-		)
-		(pin "11"
-		)
-		(pin "12"
-		)
-		(pin "13"
-		)
-		(pin "14"
-		)
-		(pin "15"
-		)
-		(pin "16"
-		)
-		(pin "17"
-		)
-		(pin "18"
-		)
-		(pin "19"
-		)
-		(pin "2"
-		)
-		(pin "20"
-		)
-		(pin "21"
-		)
-		(pin "22"
-		)
-		(pin "23"
-		)
-		(pin "24"
-		)
-		(pin "25"
-		)
-		(pin "26"
-		)
-		(pin "27"
-		)
-		(pin "28"
-		)
-		(pin "29"
-		)
-		(pin "3"
-		)
-		(pin "30"
-		)
-		(pin "31"
-		)
-		(pin "32"
-		)
-		(pin "33"
-		)
-		(pin "34"
-		)
-		(pin "35"
-		)
-		(pin "36"
-		)
-		(pin "37"
-		)
-		(pin "38"
-		)
-		(pin "39"
-		)
-		(pin "4"
-		)
-		(pin "40"
-		)
-		(pin "41"
-		)
-		(pin "42"
-		)
-		(pin "43"
-		)
-		(pin "44"
-		)
-		(pin "45"
-		)
-		(pin "46"
-		)
-		(pin "47"
-		)
-		(pin "48"
-		)
-		(pin "5"
-		)
-		(pin "6"
-		)
-		(pin "7"
-		)
-		(pin "8"
-		)
-		(pin "9"
-		)
-		(instances
-			(project "glycon"
-				(path "/956d8204-2614-4e68-9498-0bae56c4b641"
-					(reference "J3")
-					(unit 1)
-				)

Commit message: More pcb progress
Parts:
- removed R10, R14, R15, R16, R6, R9: 10K, Resistor_THT:R_Axial_DIN0207_L6.3mm_D2.5mm_P10.16mm_Horizontal, symbol Device:R
- added JP1, JP2: Jumper, Connector_PinHeader_2.54mm:PinHeader_2x01_P2.54mm_Vertical, symbol Jumper:Jumper_2_Bridged
Connections:
- net +5V: now also J2.1 (Pin_1), J3.24 (Pin_24); no longer J1.40 (Pin_40), J2.6 (Pin_6), J3.12 (Pin_12), J3.34 (Pin_34), R5.1
- net A0: now also J1.18 (Pin_18); no longer J1.3 (Pin_3)
- net A1: now also J1.17 (Pin_17); no longer J1.5 (Pin_5)
- net A10: now also J1.8 (Pin_8); no longer J1.9 (Pin_9)
- net A11: now also J1.7 (Pin_7); no longer J1.15 (Pin_15)
- net A12: now also J1.6 (Pin_6); no longer J1.29 (Pin_29)
- net A13: now also J1.5 (Pin_5); no longer J1.27 (Pin_27)
- net A14: now also J1.4 (Pin_4); no longer J1.16 (Pin_16), J1.37 (Pin_37)
- net A15: now also J1.3 (Pin_3); no longer J1.14 (Pin_14)
- net A16: now also J1.2 (Pin_2); no longer J1.12 (Pin_12)
- net A17: now also J1.1 (Pin_1)
- net A2: now also J1.16 (Pin_16); no longer J1.7 (Pin_7)
- net A3: now also J1.15 (Pin_15); no longer J1.11 (Pin_11)
- net A4: now also J1.14 (Pin_14); no longer J1.13 (Pin_13)
- net A5: now also J1.13 (Pin_13); no longer J1.17 (Pin_17)
- net A6: now also J1.12 (Pin_12); no longer J1.21 (Pin_21)
- net A7: now also J1.11 (Pin_11); no longer J1.25 (Pin_25)
- net A8: now also J1.10 (Pin_10); no longer J1.23 (Pin_23)
- net A9: now also J1.9 (Pin_9); no longer J1.19 (Pin_19)
- net ARDY: now also J3.11 (Pin_11); no longer J3.21 (Pin_21)
- net BRDY: now also J3.21 (Pin_21); no longer J3.23 (Pin_23)
- net CLK: now also J1.36 (Pin_36), J3.35 (Pin_35); no longer J1.6 (Pin_6), J3.36 (Pin_36)
- net CT1: now also J3.41 (Pin_41); no longer J3.42 (Pin_42)
- net CT2: now also J3.43 (Pin_43); no longer J3.44 (Pin_44)
- net CT3: now also J3.45 (Pin_45); no longer J3.46 (Pin_46)
- net CTSB: now also J2.3 (Pin_3); no longer J2.4 (Pin_4)
- net D0: now also J1.25 (Pin_25); no longer J1.24 (Pin_24)
- net D2: now also J1.23 (Pin_23); no longer J1.28 (Pin_28)
- net D3: now also J1.20 (Pin_20); no longer J1.30 (Pin_30)
- net D4: now also J1.19 (Pin_19); no longer J1.32 (Pin_32)
- net D5: now also J1.21 (Pin_21); no longer J1.34 (Pin_34)
- net D6: now also J1.22 (Pin_22); no longer J1.36 (Pin_36)
- net D7: now also J1.24 (Pin_24); no longer J1.38 (Pin_38)
- net Earth: now also J1.39 (Pin_39), J2.2 (Pin_2), J3.23 (Pin_23); no longer J1.1 (Pin_1), J2.5 (Pin_5), J3.11 (Pin_11), J3.33 (Pin_33)
- net PA0: now also J3.9 (Pin_9); no longer J3.19 (Pin_19)
- net PA1: now also J3.10 (Pin_10); no longer J3.20 (Pin_20)
- net PA2: now also J3.7 (Pin_7); no longer J3.17 (Pin_17)
- net PA3: now also J3.8 (Pin_8); no longer J3.18 (Pin_18)
- net PA4: now also J3.5 (Pin_5); no longer J3.15 (Pin_15)
- net PA5: now also J3.6 (Pin_6); no longer J3.16 (Pin_16)
- net PA6: now also J3.3 (Pin_3); no longer J3.13 (Pin_13)
- net PA7: now also J3.4 (Pin_4); no longer J3.14 (Pin_14)
- net PB0: now also J3.19 (Pin_19); no longer J3.26 (Pin_26)
- net PB1: now also J3.20 (Pin_20); no longer J3.25 (Pin_25)
- net PB2: now also J3.17 (Pin_17); no longer J3.28 (Pin_28)
- net PB3: now also J3.18 (Pin_18); no longer J3.27 (Pin_27)
- net PB4: now also J3.15 (Pin_15); no longer J3.30 (Pin_30)
- net PB5: now also J3.16 (Pin_16); no longer J3.29 (Pin_29)
- net PB6: now also J3.13 (Pin_13); no longer J3.32 (Pin_32)
- net PB7: now also J3.14 (Pin_14); no longer J3.31 (Pin_31)
- net PC0: no longer J3.35 (Pin_35)
- net PC1: no longer J3.37 (Pin_37)
- net PC2: no longer J3.39 (Pin_39)
- net PC3: no longer J3.41 (Pin_41)
- net PGA0: no longer J1.31 (Pin_31)
- net PGA1: no longer J1.33 (Pin_33)
- net RAM WE: now also J1.35 (Pin_35); no longer J1.22 (Pin_22)
- net RAM/ROM OE: now also J1.37 (Pin_37); no longer J1.20 (Pin_20)
- net RTSB: now also J2.6 (Pin_6); no longer J2.1 (Pin_1)
- net RXDA: now also J3.28 (Pin_28); no longer J3.3 (Pin_3)
- net RxDB: now also J2.5 (Pin_5); no longer J2.2 (Pin_2)
- net SERCLK: now also JP1.1 (A); no longer U7.13 (~{RXCA}), U7.14 (~{TXCA})
- net SYNCA: now also J3.25 (Pin_25); no longer J3.5 (Pin_5)
- net TO1: now also J3.37 (Pin_37); no longer J3.38 (Pin_38)
- net TO2: now also J3.39 (Pin_39); no longer J3.40 (Pin_40)
- net TXDA: now also J3.27 (Pin_27); no longer J3.9 (Pin_9)
- net TxDB: now also J2.4 (Pin_4); no longer J2.3 (Pin_3)
- net VDD: now also J1.40 (Pin_40), R3.1, R5.2; no longer R3.2, U0.24 (~{WAIT})
- net ~{ASTB}: now also J3.12 (Pin_12); no longer J3.22 (Pin_22)
- net ~{BSTB}: now also J3.22 (Pin_22); no longer J3.24 (Pin_24)
- net ~{BUSACK}: now also J1.30 (Pin_30); no longer J1.10 (Pin_10)
- net ~{BUSRQ}: now also J1.28 (Pin_28), R2.1; no longer J1.35 (Pin_35)
- net ~{CTSA}: now also J3.32 (Pin_32); no longer J3.8 (Pin_8)
- net ~{DCDA}: now also J3.31 (Pin_31); no longer J3.4 (Pin_4)
- net ~{DTRA}: now also J3.30 (Pin_30); no longer J3.6 (Pin_6)
- net ~{INT}: now also J1.29 (Pin_29); no longer J1.39 (Pin_39)
- net ~{IORQ}: no longer J1.18 (Pin_18)
- net ~{IO_RD}: no longer R2.1
- net ~{M1}: now also J1.31 (Pin_31); no longer J1.8 (Pin_8)
- net ~{RESET}: now also J1.27 (Pin_27)
- net ~{ROM_WE}: now also J1.38 (Pin_38), R3.2; no longer J1.2 (Pin_2), R5.2
- net ~{RTSA}: now also J3.29 (Pin_29); no longer J3.10 (Pin_10)
- net ~{Z80_WR}: no longer R3.1
- net ~{WAIT}: now reaches U7.30 (~{W}/~{RDYB})
- net ~{WAIT}: now also R5.1, U0.24 (~{WAIT}), U7.10 (~{W}/~{RDYA})
- removed net RESET: J1.4 (Pin_4), J3.43 (Pin_43)
- removed net ~{W}/~{RDYA}: J3.7 (Pin_7), U7.10 (~{W}/~{RDYA})
- new net: JP2.2 (B), U7.13 (~{RXCA})
- new net: JP1.2 (B), JP2.1 (A), U7.14 (~{TXCA})
- no-connect marks 16 -> 14

Commit message: almost finalized new pcb design
Parts:
- renumbered IC2 to U12
Connections:
- net +5V: now also J2.3 (Pin_3), J3.34 (Pin_34); no longer J2.1 (Pin_1)
- net CLK: now also X1.5 (OUT); no longer X1.8 (OUT)
- net Earth: now also J2.1 (Pin_1), J3.33 (Pin_33), X1.4 (GND); no longer J2.2 (Pin_2), X1.7 (GND)
- net PC0: now also J3.36 (Pin_36)
- net PC1: now also J3.38 (Pin_38)
- net PC2: now also J3.40 (Pin_40)
- net PC3: now also J3.42 (Pin_42)
- net VDD: now also X1.8 (Vcc); no longer X1.14 (Vcc)
- net CTSB renamed ~{CTSB}
- net ~{CTSB}: now also J2.2 (Pin_2); no longer J2.3 (Pin_3)
- net RTSB renamed ~{RTSB}
